File: subprojects/external-iv9-socket/external-iv9-socket.kicad_pcb (KiCad board)
At the start: 2 copper layers, 20.1 x 15.1 mm, 3 parts, among them J1 PINHD_1x5_Male, J3 PINHD_1x4_Male

Commit message: Veľké pokroky pri navrhu DPS.
Parts:
- J1: value PINHD_1x5_Male -> PINHD_1x6_Male; footprint Connector_PinHeader_2.54mm:PinHeader_1x05_P2.54mm_Vertical -> Connector_PinHeader_2.54mm:PinHeader_1x06_P2.54mm_Vertical
- U$1: footprint VacuumTubes:IV-9 -> VacuumTubes:IV-9-Common-Separated
- moved J1 19.3 mm to (108.5, 81.7), turned to 0 degrees
- moved J3 14.7 mm to (94.2, 69.0)
- turned U$1 to 0 degrees
Connections:
- J1 pad 2: Net-(J1-Pad2) -> unconnected-(J1-Pad2)
- U$1 pad 2: Net-(J3-Pad1) -> Net-(J1-Pad3)
- U$1 pad 3: Net-(J3-Pad2) -> Net-(J1-Pad4)
- U$1 pad 4: Net-(J3-Pad3) -> Net-(J1-Pad5)
- U$1 pad 5: Net-(J3-Pad4) -> Net-(J1-Pad6)
- U$1 pad 6: Net-(J1-Pad5) -> Net-(J3-Pad1)
- U$1 pad 7: Net-(J1-Pad4) -> Net-(J3-Pad2)
- U$1 pad 8: Net-(J1-Pad3) -> Net-(J3-Pad3)
- U$1 pad 9: Net-(J1-Pad2) -> Net-(J3-Pad4)
Routing:
- net Net-(J1-Pad6): track 0.00 -> 8.26 mm
- net Net-(J1-Pad2): track 5.79 -> 0.00 mm
- net Net-(J3-Pad4): track 8.53 -> 5.61 mm
- net Net-(J1-Pad1): track 9.81 -> 7.91 mm
- net Net-(J3-Pad3): track 6.80 -> 5.34 mm
- net Net-(J3-Pad2): track 6.06 -> 5.10 mm
- net Net-(J1-Pad5): track 6.86 -> 5.91 mm
- net Net-(J1-Pad4): track 5.29 -> 4.68 mm
Other:
- board size 20.1 x 15.1 mm -> 17.8 x 16.3 mm

Commit message: Pomerne velke zmeny a prehodnotenia zakladnych veci.
Parts:
- moved U$1 1.49 mm to (101.3, 72.8)
Routing:
- net Net-(J3-Pad3): track 5.34 -> 4.23 mm
- net Net-(J3-Pad2): track 5.10 -> 4.23 mm
- net Net-(J3-Pad1): track 6.65 -> 5.78 mm
- net Net-(J1-Pad1): track 7.91 -> 8.55 mm
Changed lines of the file:
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@@
 	(net 8 "Net-(J3-Pad3)")
 	(net 9 "Net-(J1-Pad6)")
-	(net 10 "unconnected-(J1-Pad2)")
 	(footprint "VacuumTubes:IV-9-Common-Separated"
 		(layer "F.Cu")
-		(at 101.366 74.295)
+		(at 101.346 72.81)
 		(descr "IV-9 Numitron")
 		(property "Reference" "U$1"
@@
 			(unlocked yes)
 			(layer "F.SilkS")
+			(hide yes)
 			(effects
 				(font
@@
 			(layer "B.Fab")
 		)
-		(fp_text user "${REFERENCE}"
-			(at 0 -3.81 90)
-			(layer "B.Fab")
-			(effects
-				(font
-					(size 1 1)
-					(thickness 0.15)
-				)
-				(justify mirror)
-			)
-		)
 		(pad "1" thru_hole circle
 			(at 0 0 180)
@@
 			(at 0 2.38 180)
 			(layer "B.SilkS")
+			(hide yes)
 			(effects
 				(font
@@
 			(layer "B.Fab")
 		)
-		(fp_text user "${REFERENCE}"
-			(at 0 -6.35 270)
-			(layer "B.Fab")
-			(effects
-				(font
-					(size 1 1)
-					(thickness 0.15)
-				)
-				(justify mirror)
-			)
-		)
 		(pad "1" thru_hole rect
 			(at 0 0)
@@
 			(net 3 "Net-(J1-Pad1)")
 			(pintype "passive")
-		)
-		(pad "2" thru_hole circle
-			(at 0 -2.54)
-			(size 1.7 1.7)
-			(drill 1)
-			(layers "*.Cu" "*.Mask")
-			(remove_unused_layers no)
-			(net 10 "unconnected-(J1-Pad2)")
-			(pintype "passive+no_connect")
 		)
 		(pad "3" thru_hole circle
@@
 	)
 	(segment
-		(start 107.4008 75.2698)
-		(end 108.736 76.605)
+		(start 105.6648 73.7848)
+		(end 104.346 73.7848)
 		(width 0.508)
 		(layer "F.Cu")
@@
 	)
 	(segment
-		(start 104.366 75.2698)
-		(end 107.4008 75.2698)
+		(start 108.5 76.62)
+		(end 105.6648 73.7848)
 		(width 0.508)
 		(layer "F.Cu")
@@
 	)
 	(segment
-		(start 103.4381 71.525)
-		(end 103.2201 71.743)
+		(start 107.218 70.258)
+		(end 103.2001 70.258)
 		(width 0.508)
 		(layer "F.Cu")
@@
 	)
 	(segment
-		(start 103.2201 71.743)
-		(end 108.518 71.743)
+		(start 108.5 71.54)
+		(end 107.218 70.258)
 		(width 0.508)
 		(layer "F.Cu")
@@
 	)
 	(segment
-		(start 108.518 71.743)
-		(end 108.736 71.525)
-		(width 0.508)
-		(layer "F.Cu")
-		(net 2)
-	)
-	(segment
-		(start 106.996 81.7)
-		(end 108.5 81.7)
+		(start 108.461 81.7)
+		(end 102.446 75.685)
 		(width 0.508)
 		(layer "F.Cu")
@@
 	)
 	(segment
-		(start 102.466 77.17)
-		(end 106.996 81.7)
+		(start 108.5 81.7)
+		(end 108.461 81.7)
 		(width 0.508)
 		(layer "F.Cu")
@@
 	)
 	(segment
-		(start 107.9912 73.3202)
-		(end 108.736 74.065)
+		(start 108.5 74.08)
+		(end 106.2552 71.8352)
 		(width 0.508)
 		(layer "F.Cu")
@@
 	)
 	(segment
-		(start 104.366 73.3202)
-		(end 107.9912 73.3202)
+		(start 106.2552 71.8352)
+		(end 104.346 71.8352)
 		(width 0.508)
 		(layer "F.Cu")
@@
 	)
 	(segment
-		(start 95.7152 73.3202)
-		(end 98.366 73.3202)
+		(start 94.234 71.54)
+		(end 98.0508 71.54)
 		(width 0.508)
 		(layer "F.Cu")
@@
 	)
 	(segment
-		(start 93.98 71.585)
-		(end 95.7152 73.3202)
+		(start 98.0508 71.54)
+		(end 98.346 71.8352)
 		(width 0.508)
 		(layer "F.Cu")
@@
 	)
 	(segment
-		(start 93.98 69.045)
-		(end 96.678 71.743)
+		(start 98.21 69)
+		(end 99.468 70.258)
 		(width 0.508)
 		(layer "F.Cu")
@@
 	)
 	(segment
-		(start 96.678 71.743)
-		(end 99.5119 71.743)
+		(start 99.468 70.258)
+		(end 99.4919 70.258)
 		(width 0.508)
 		(layer "F.Cu")
@@
 	)
 	(segment
-		(start 93.98 76.665)
-		(end 94.162 76.847)
+		(start 94.234 69)
+		(end 98.21 69)
+		(width 0.508)
+		(layer "F.Cu")
+		(net 6)
+	)
+	(segment
+		(start 94.234 76.62)
+		(end 98.2339 76.62)
 		(width 0.508)
 		(layer "F.Cu")
@@
 	)
 	(segment
-		(start 94.162 76.847)
-		(end 99.5119 76.847)
+		(start 98.2339 76.62)
+		(end 99.4919 75.362)
 		(width 0.508)
 		(layer "F.Cu")
@@
 	)
 	(segment
-		(start 95.1248 75.2698)
-		(end 98.366 75.2698)
+		(start 98.0508 74.08)
+		(end 98.346 73.7848)
 		(width 0.508)
 		(layer "F.Cu")
@@
 	)
 	(segment
-		(start 98.0262 74.93)
-		(end 98.366 75.2698)
+		(start 94.234 74.08)
+		(end 98.0508 74.08)
 		(width 0.508)
 		(layer "F.Cu")
@@
 	)
 	(segment
-		(start 93.98 74.125)
-		(end 95.1248 75.2698)
-		(width 0.508)
-		(layer "F.Cu")
-		(net 8)
-	)
-	(segment
-		(start 101.366 71.1406)
-		(end 103.5216 68.985)
+		(start 107.65 68.15)
+		(end 102.8516 68.15)
 		(width 0.508)
 		(layer "F.Cu")
@@
 	)
 	(segment
-		(start 103.5216 68.985)
-		(end 108.736 68.985)
-		(width 0.508)
-		(layer "F.Cu")
+		(start 102.8516 68.15)
+		(end 101.346 69.6556)
+		(width 0.508)
+		(layer "F.Cu")
+		(net 9)
+	)
+	(segment
+		(start 108.5 69)
+		(end 107.65 68.15)
+		(width 0.508)
+		(layer "F.Cu")

Commit message: preventivne
Routing:
- net Net-(J1-Pad1): track 8.55 -> 0.00 mm
- net Net-(J1-Pad4): track 5.08 -> 3.38 mm
- net Net-(J1-Pad5): track 5.90 -> 4.52 mm
- net Net-(J1-Pad3): track 5.33 -> 4.20 mm
- net Net-(J1-Pad6): track 7.75 -> 6.64 mm

Commit message: Prvá iterácia.
Routing:
- net Net-(J1-Pad1): track 0.00 -> 12.4 mm
- net Net-(J3-Pad1): track 5.78 -> 9.54 mm
- net Net-(J3-Pad2): track 4.23 -> 6.51 mm
- net Net-(J1-Pad3): track 4.20 -> 5.97 mm
- net Net-(J1-Pad4): track 3.38 -> 4.53 mm
- net Net-(J3-Pad3): track 4.23 -> 5.11 mm
- net Net-(J1-Pad6): track 6.64 -> 6.00 mm
Other:
- board size 17.8 x 16.3 mm -> 17.8 x 17.2 mm

Commit message: Zase po dlhšej dobe preventívny commit.
Parts:
- removed J1: PINHD_1x6_Male, Connector_PinHeader_2.54mm:PinHeader_1x06_P2.54mm_Vertical
- added REF**: PinHeader_1x06_P2.54mm_Vertical, Connector_PinHeader_2.54mm:PinHeader_1x06_P2.54mm_Vertical, B.Cu at (114.0, 57.5)
- moved J3 24.8 mm to (99.7, 44.8)
- moved U$1 24.8 mm to (106.8, 48.6)

Commit message: Pridaný firmware.
Parts:
- removed REF**: PinHeader_1x06_P2.54mm_Vertical, Connector_PinHeader_2.54mm:PinHeader_1x06_P2.54mm_Vertical
- added J1: PINHD_1x6_Male, Connector_PinHeader_2.54mm:PinHeader_1x06_P2.54mm_Vertical, F.Cu at (114.0, 57.5)
Other:
- board size 17.8 x 17.2 mm -> 17.8 x 18 mm
