File: numeri-iv9-hodiny.kicad_sch (KiCad schematic)
At the start: 57 parts, among them J1 USB-C, J3 2x3, J5 USB_C_Receptacle_PowerOnly_6P, Q1 BC547, SW1 RESET, SW2 Horizontal, SW3 Vertical, U1 LM2596T-5, U2 ATtiny24A-PU, U3 TPIC6B595N, Y1 6MHz

Commit message: Pridaný kód firmwaru + úpravy schéma a DPS s anglickým prekladom.
Parts:
- removed C16, C17: 100n, Capacitor_THT:C_Disc_D3.0mm_W2.0mm_P2.50mm, symbol PCM_SL_Devices:Capacitor_NP
- removed DCF-3850N-1: DCF77, Connector_PinHeader_2.54mm:PinHeader_1x04_P2.54mm_Vertical, symbol Numitronové_hodiny_v12-eagle-import:con-amp-quick_125_M04
- removed F1: F1.25A/250VDC, Fuse:Fuseholder_Cylinder-5x20mm_Schurter_0031_8201_Horizontal_Open, symbol Numitronové_hodiny_v12-eagle-import:fuse_233_SHK20L
- removed H_:__1, _H:__1, __:M_1, __:_M1: IV-9, Connector_PinSocket_2.54mm:PinSocket_1x04_P2.54mm_Vertical, symbol Numitronové_hodiny_v12-eagle-import:domestichacks_IV-9
- removed Q1: BC547, Package_TO_SOT_THT:TO-92_Inline, symbol Transistor_BJT:BC547
- removed R10, R2, R4: 10k, Resistor_THT:R_Axial_DIN0207_L6.3mm_D2.5mm_P10.16mm_Horizontal, symbol PCM_SL_Resistors:Resistor
- removed SW1: RESET, Button_Switch_THT:SW_PUSH_6mm, symbol PCM_SL_Devices:Push_Button
- removed TVS1: P6KE250A, Diode_THT:D_DO-41_SOD81_P10.16mm_Horizontal, symbol Diode:1N4005
- removed U2: ATtiny24A-PU, Package_DIP:DIP-14_W7.62mm_Socket, symbol MCU_Microchip_ATtiny:ATtiny24A-P
- removed U3: TPIC6B595N, Package_DIP:DIP-20_W7.62mm_Socket, symbol hodiny-eagle-import:TPIC6B595N
- removed U4, U5, U6: ~, Package_DIP:DIP-20_W7.62mm_Socket, symbol hodiny-eagle-import:TPIC6B595N
- added C13, C14: 100n, Capacitor_THT:C_Disc_D3.0mm_W2.0mm_P2.50mm, symbol PCM_SL_Devices:Capacitor_NP
- added DCF-3850N-1: DCF77, Connector_PinHeader_2.54mm:PinHeader_1x04_P2.54mm_Vertical, symbol DCF77_Module_DCF-3850N-1:con-amp-quick_125_M04
- added F1: F1.25A, Fuse:Fuseholder_Cylinder-5x20mm_Schurter_0031_8201_Horizontal_Open, symbol Device:Fuse
- added H1: IV-9, Connector_PinHeader_1.00mm:PinHeader_1x05_P1.00mm_Vertical, symbol VacuumTubes:IV-9
- added H2, M1, M2: IV-9, VacuumTubes:IV-9, symbol VacuumTubes:IV-9
- added R11: 1K5, Resistor_THT:R_Axial_DIN0207_L6.3mm_D2.5mm_P10.16mm_Horizontal, symbol PCM_SL_Resistors:Resistor
- added R7: 10K, Resistor_THT:R_Axial_DIN0207_L6.3mm_D2.5mm_P10.16mm_Horizontal, symbol PCM_SL_Resistors:Resistor
- added TSV1: BZW06-5V8, Diode_THT:D_DO-201AE_P15.24mm_Horizontal, symbol Diode:1N62xxA
- added U2: ATtiny24A-PU, Package_DIP:DIP-14_W7.62mm_Socket, symbol ATtinyx4A-PU:ATtiny24A-P
- added U3, U4, U5, U6: TPIC6B595N, Package_DIP:DIP-20_W7.62mm_Socket, symbol SIPO_Register_TPIC6B595N:TPIC6B595N
- C1: renamed from C2; value 470uF_25V -> 470uF; Voltage (none) -> 10V
- C17: renamed from C12; value 100n -> 100nF
- C2: renamed from C6; value 470uF_10V -> 470uF; Voltage (none) -> 10V
- R1: renamed from R12; value 5.1k -> 5K1
- R10: renamed from R3; value 10k -> 2K5
- R2: renamed from R13; value 5.1k -> 5K1
- R3: renamed from R11; value 10k -> 10K
- R4: renamed from R5; value 10k -> 10K
- R5: renamed from R6; value 10k -> 10K
- R6: renamed from R7; value 10k -> 10K
- R8, R9: value 10k -> 10K
- renumbered C11 to C10, C13 to C11, C14 to C12, C9 to C16, C1 to C6, C10 to C9, D6 to D1, D8 to D2, D7 to D3, J5 to J1, J1 to J2, L2 to L1, SW2 to SW1, SW3 to SW2
Connections:
- net PA5 is gone; now on net ~PA5/MISO: R4.1
- net +5VBAT: now also U2.1 (VCC)
- net +5VREG: now also C1.1, C2.1, U1.1 (VIN), C13.2, C14.2, F1.2, H1.1, H2.1, M1.1, M2.1, R7.2, TSV1.1 (A1), U3.2 (VCC), U4.2 (VCC), U5.2 (VCC), U6.2 (VCC); no longer C2.2
- net GND: now also C2.2, C13.1, C14.1, DCF-3850N-1.2 (GND), TSV1.2 (A2), U2.14 (GND), U3.10 (GND_2), U3.11 (GND), U3.19 (GND_3), U4.10 (GND_2), U4.11 (GND), U4.19 (GND_3), U5.10 (GND_2), U5.11 (GND), U5.19 (GND_3), U6.10 (GND_2), U6.11 (GND), U6.19 (GND_3); no longer C2.1
- net P2: now also H2.2, M1.2, M2.2, U4.4 (DRAIN0), U5.4 (DRAIN0), U6.4 (DRAIN0)
- net P3: now also H2.3, M1.3, M2.3, U4.5 (DRAIN1), U5.5 (DRAIN1), U6.5 (DRAIN1)
- net P4: now also H2.4, M1.4, M2.4, U3.6 (DRAIN2), U4.6 (DRAIN2), U5.6 (DRAIN2), U6.6 (DRAIN2)
- net P5: now also H1.5, H2.5, M1.5, M2.5, U3.7 (DRAIN3), U4.7 (DRAIN3), U5.7 (DRAIN3), U6.7 (DRAIN3)
- net P6: now also H1.6, H2.6, M1.6, M2.6, U3.14 (DRAIN4), U4.14 (DRAIN4), U5.14 (DRAIN4), U6.14 (DRAIN4)
- net P7: now also H1.7, H2.7, M1.7, M2.7, U3.15 (DRAIN5), U4.15 (DRAIN5), U5.15 (DRAIN5), U6.15 (DRAIN5)
- net P8: now also H1.8, H2.8, M1.8, M2.8, U3.16 (DRAIN6), U4.16 (DRAIN6), U5.16 (DRAIN6), U6.16 (DRAIN6)
- net P9: now also H2.9, M1.9, M2.9, U3.17 (DRAIN7), U4.17 (DRAIN7), U5.17 (DRAIN7), U6.17 (DRAIN7)
- net PA2: now also U2.11 (PA2), U3.3 (SER_IN)
- net PA3: now also U2.10 (PA3), U3.13 (SRCK), U4.13 (SRCK), U5.13 (SRCK), U6.13 (SRCK)
- net PA4/SCL: now also U2.9 (SCL/PA4), U3.12 (RCK), U4.12 (RCK), U5.12 (RCK), U6.12 (RCK)
- net VCC: now also F1.1
- net ~PA5/MISO: now also U2.8 (MISO/PA5~)
- net ~PA6/MOSI/SDA: now also U2.7 (SDA/MOSI/PA6~), U3.9 (~{G}), U4.9 (~{G}), U5.9 (~{G}), U6.9 (~{G})
- net at D5.2: now also R11.1
- net at C16.1, C17.2, D4.1 (K)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: now also DCF-3850N-1.1 (VCC)
- net at C10.2, SW1.1: now also U2.5 (INT0/PB2~)
- net at C7.2, Y1.1: now also U2.2 (PB0/XTAL1)
- net at C8.2, Y1.2: now also U2.3 (PB1/XTAL2)
- net at C11.2, SW2.1: now also U2.6 (PA7~)
- net at R6.1: now also U3.8 (~{SRCLR})
- net at R9.1: now also U6.8 (~{SRCLR})
- net at R8.1: now also U5.8 (~{SRCLR})
- net ~{RESET}/PB3 renamed ~{RESET}
- net ~{RESET}: now also U2.4 (PB3/~{RESET})
- new net: U3.18 (SER_OUT), U4.3 (SER_IN)
- new net: U5.18 (SER_OUT), U6.3 (SER_IN)
- new net: U4.18 (SER_OUT), U5.3 (SER_IN)
- new net: R7.1, U4.8 (~{SRCLR})
- new net H1_2: H1.2, U3.4 (DRAIN0)
- new net H1_3: H1.3, U3.5 (DRAIN1)
- new net H1_4: H1.4
- new net H1_9: H1.9
- new net PA0: DCF-3850N-1.3 (OUT), R11.2, U2.13 (AREF/PA0)
- new net PA1: DCF-3850N-1.4 (~{PON}), U2.12 (PA1)
Other:
- note added: "I = 5V / 10K = 500uA P = 5V * 500uA = 2,5mW"
- note added: "Napájací zdroj"
- note added: "Nemusíme upravovat logiku, použijeme ADC prevodník."
- note added: "Poistka môže byť aj na panely."
- note added: "R = 5V/2mA = 2K5"
- note added: "Toto by bolo dobré mať zapojené v sérii (x1R), problém je ale referenčný bod. Nevieme koľko tam bolo nazačiatku, takže ťažko povedať koľko tam je teraz."
- note added: "~ marks a PWM pin"
- note removed: "Bez USB-PD vieme dostať napätie do 5V."
- note removed: "I = 5V / 10k = 500uA P = 5V * 500uA = 2,5mW"
- note removed: "R = 5V/2.5mA = 2k"
- note removed: "R = 5V/2mA = 2,5k"
- note removed: "Vnútorný napájací zdroj"
- moved on the sheet: C10, C11, C12, C16, C17, C2, C7, C8, C9, D4, D5, J3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

Commit message: Veľké pokroky pri navrhu DPS.
Parts:
- removed C2: 470uF, Capacitor_THT:CP_Radial_D8.0mm_P3.50mm, symbol PCM_SL_Capacitors:470uF_10V
- removed C3, C4: 1000uF, Capacitor_THT:CP_Radial_D10.0mm_P5.00mm, symbol PCM_SL_Capacitors:1000uF_16V
- removed D1: 1N5817, Diode_THT:D_DO-41_SOD81_P10.16mm_Horizontal, symbol Diode:1N5817
- removed L1: 33uH, Inductor_THT:L_CommonMode_Toroid_Vertical_L19.3mm_W10.8mm_Px6.35mm_Py15.24mm_Bourns_8100, symbol Device:L
- removed R4: 10K, Resistor_THT:R_Axial_DIN0207_L6.3mm_D2.5mm_P10.16mm_Horizontal, symbol PCM_SL_Resistors:Resistor
- removed U1: LM2596T-5, Package_TO_SOT_THT:TO-220-5_P3.4x3.7mm_StaggerOdd_Lead3.8mm_Vertical, symbol Regulator_Switching:LM2596T-5
- added R12: 10K, Resistor_THT:R_Axial_DIN0207_L6.3mm_D2.5mm_P10.16mm_Horizontal, symbol PCM_SL_Resistors:Resistor
- C1: value 470uF -> 4,7uF
- C12, C13, C14, C15: value 100n -> 100nF
- C6: value 100uF -> 3,3uF
- D2, D3: value 1N5817 -> 1N5822
- D5: footprint LED_THT:LED_D5.0mm -> TerminalBlock_Phoenix:TerminalBlock_Phoenix_MPT-0,5-2-2.54_1x02_P2.54mm_Horizontal
- DCF-3850N-1: footprint Connector_PinHeader_2.54mm:PinHeader_1x04_P2.54mm_Vertical -> Connector_PinSocket_2.54mm:PinSocket_1x04_P2.54mm_Vertical
- H1: footprint Connector_PinHeader_1.00mm:PinHeader_1x05_P1.00mm_Vertical -> VacuumTubes:IV-9_External_Socket_Asymetric
- H2, M1, M2: footprint VacuumTubes:IV-9 -> VacuumTubes:IV-9_External_Socket_Asymetric
- SW1, SW2: footprint TerminalBlock_Phoenix:TerminalBlock_Phoenix_MKDS-1,5-2_1x02_P5.00mm_Horizontal -> TerminalBlock_Phoenix:TerminalBlock_Phoenix_MPT-0,5-2-2.54_1x02_P2.54mm_Horizontal
Connections:
- net ~PA5/MISO is gone; now on net MISO/HBTN: J3.6, U2.8 (MISO/PA5~)
- net +5VREG: now also R12.2
- net H1_4: now also U3.6 (DRAIN2)
- net H1_9: now also U3.17 (DRAIN7)
- net +3.3V: now reaches C16.1, C17.2, D4.1 (K), DCF-3850N-1.1 (VCC), R10.1
- net MISO/HBTN: now reaches C10.2, SW1.1
- net MISO/HBTN: no longer U2.5 (INT0/PB2~)
- net VBTN: now reaches C11.2, SW2.1
- net VBTN: now also U2.10 (PA3); no longer U2.6 (PA7~)
- removed net P2: H2.2, M1.2, M2.2, U4.4 (DRAIN0), U5.4 (DRAIN0), U6.4 (DRAIN0)
- removed net P3: H2.3, M1.3, M2.3, U4.5 (DRAIN1), U5.5 (DRAIN1), U6.5 (DRAIN1)
- removed net P4: H2.4, M1.4, M2.4, U3.6 (DRAIN2), U4.6 (DRAIN2), U5.6 (DRAIN2), U6.6 (DRAIN2)
- removed net P5: H1.5, H2.5, M1.5, M2.5, U3.7 (DRAIN3), U4.7 (DRAIN3), U5.7 (DRAIN3), U6.7 (DRAIN3)
- removed net P6: H1.6, H2.6, M1.6, M2.6, U3.14 (DRAIN4), U4.14 (DRAIN4), U5.14 (DRAIN4), U6.14 (DRAIN4)
- removed net P7: H1.7, H2.7, M1.7, M2.7, U3.15 (DRAIN5), U4.15 (DRAIN5), U5.15 (DRAIN5), U6.15 (DRAIN5)
- removed net P8: H1.8, H2.8, M1.8, M2.8, U3.16 (DRAIN6), U4.16 (DRAIN6), U5.16 (DRAIN6), U6.16 (DRAIN6)
- removed net P9: H2.9, M1.9, M2.9, U3.17 (DRAIN7), U4.17 (DRAIN7), U5.17 (DRAIN7), U6.17 (DRAIN7)
- net PA0 renamed OUT
- net PA1 renamed ~{PON}
- net PA2 renamed SER_IN
- net PA3 renamed MOSI/SRCK
- net MOSI/SRCK: now also J3.5, U2.7 (SDA/MOSI/PA6~); no longer U2.10 (PA3)
- net PA4/SCL renamed RCK
- net RCK: now also U2.6 (PA7~); no longer J3.4, U2.9 (SCL/PA4)
- net ~PA6/MOSI/SDA renamed ~{G}~
- net ~{G}~: now also U2.5 (INT0/PB2~); no longer J3.5, U2.7 (SDA/MOSI/PA6~)
- new net ADC/SCL: J3.4, R12.1, U2.9 (SCL/PA4)
- new net H1_5: H1.5, U3.7 (DRAIN3)
- new net H1_6: H1.6, U3.14 (DRAIN4)
- new net H1_7: H1.7, U3.15 (DRAIN5)
- new net H1_8: H1.8, U3.16 (DRAIN6)
- new net H2_2: H2.2, U4.4 (DRAIN0)
- new net H2_3: H2.3, U4.5 (DRAIN1)
- new net H2_4: H2.4, U4.6 (DRAIN2)
- new net H2_5: H2.5, U4.7 (DRAIN3)
- new net H2_6: H2.6, U4.14 (DRAIN4)
- new net H2_7: H2.7, U4.15 (DRAIN5)
- new net H2_8: H2.8, U4.16 (DRAIN6)
- new net H2_9: H2.9, U4.17 (DRAIN7)
- new net M1_2: M1.2, U5.4 (DRAIN0)
- new net M1_3: M1.3, U5.5 (DRAIN1)
- new net M1_4: M1.4, U5.6 (DRAIN2)
- new net M1_5: M1.5, U5.7 (DRAIN3)
- new net M1_6: M1.6, U5.14 (DRAIN4)
- new net M1_7: M1.7, U5.15 (DRAIN5)
- new net M1_8: M1.8, U5.16 (DRAIN6)
- new net M1_9: M1.9, U5.17 (DRAIN7)
- new net M2_2: M2.2, U6.4 (DRAIN0)
- new net M2_3: M2.3, U6.5 (DRAIN1)
- new net M2_4: M2.4, U6.6 (DRAIN2)
- new net M2_5: M2.5, U6.7 (DRAIN3)
- new net M2_6: M2.6, U6.14 (DRAIN4)
- new net M2_7: M2.7, U6.15 (DRAIN5)
- new net M2_8: M2.8, U6.16 (DRAIN6)
- new net M2_9: M2.9, U6.17 (DRAIN7)
Other:
- note added: ""Bleeding" resistor for discharging the capacitors when power is switched off."
- note added: "Atomic clock signal receiver"
- note added: "Battery backup"
- note added: "Brightness regulation (PWM)"
- note added: "Detekcia napájania"
- note added: "MCU + Controls"
- note added: "Numitron Display (4xIV-9)"
- note added: "Panel mount power connector - USB Type C"
- note added: "Power supply"
- note added: "Programming bus for the MCU"
- note added: "Screw terminal for VBUS and GND from the USB-C receptacle."
- note added: "The fuse can be on the case as well."
- note removed: "* PWM piny"
- note removed: "Detekcia napájania zo siete."
- note removed: "MCU + Ovládanie"
- note removed: "Napájací konektor - USB Typ C"
- note removed: "Napájací zdroj"
- note removed: "Nemusíme upravovat logiku, použijeme ADC prevodník."
- note removed: "Numitronový displej (4xIV-9)"
- note removed: "Poistka môže byť aj na panely."
- note removed: "Prijímač signálu atómových hodín"
- note removed: "Pull-up rezistor zaisťuje, že registre ostanú vypnuté ak odíde mikrokontróler."
- note removed: "Regulácia jasu (PWM)"
- note removed: "Toto by bolo dobré mať zapojené v sérii (x1R), problém je ale referenčný bod. Nevieme koľko tam bolo nazačiatku, takže ťažko povedať koľko tam je teraz."
- note removed: "USB-C konektor na panely nám umožní pridať vypínač bez úprav dosky."
- note removed: "Zbernica pre programovanie MCU"
- note removed: "Záložné napájanie"
- company: Filip Mitka -> (none)
- title: Numitronové Hodiny -> Numitron Clock with DCF77
- moved on the sheet: BT1, C1, C10, C11, C16, C17, C5, C6, D2, D3, D4, D5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

Commit message: Pomerne velke zmeny a prehodnotenia zakladnych veci.
Parts:
- removed C1: 4,7uF, Capacitor_THT:CP_Radial_D8.0mm_P3.50mm, symbol PCM_SL_Capacitors:470uF_25V
- removed R11: 1K5, Resistor_THT:R_Axial_DIN0207_L6.3mm_D2.5mm_P10.16mm_Horizontal, symbol PCM_SL_Resistors:Resistor
- added C2: 4.7uF, Capacitor_THT:CP_Radial_D5.0mm_P2.00mm, symbol PCM_SL_Capacitors:4.7uF_16V
- added EM2S1, MASD-S-R1: DCF77, Connector_PinSocket_2.54mm:PinSocket_1x04_P2.54mm_Vertical, symbol DCF77_Module_DCF-3850N-1:con-amp-quick_125_M04
- added R13: 10K, Resistor_THT:R_Axial_DIN0207_L6.3mm_D2.5mm_P5.08mm_Vertical, symbol PCM_SL_Resistors:Resistor
- added R4: 50K, PCM_SL_Devices:potentiometer_3362P, symbol Device:R_Trim
- added TSV2: BZW06-5V8, Diode_THT:D_DO-201AE_P15.24mm_Horizontal, symbol Diode:1N62xxA
- R12, R5: footprint Resistor_THT:R_Axial_DIN0207_L6.3mm_D2.5mm_P10.16mm_Horizontal -> Resistor_THT:R_Axial_DIN0207_L6.3mm_D2.5mm_P5.08mm_Vertical
- R3: footprint Resistor_THT:R_Axial_DIN0207_L6.3mm_D2.5mm_P10.16mm_Horizontal -> Resistor_THT:R_Axial_DIN0207_L6.3mm_D2.5mm_P2.54mm_Vertical
Connections:
- net +3.3V: now also MASD-S-R1.1 (VCC)
- net +5VBAT: now also J3.5, R13.2; no longer J3.1
- net +5VREG: now also C2.1, EM2S1.1 (VCC), TSV2.1 (A1)
- net GND: now also J3.1, C2.2, EM2S1.4 (GND), MASD-S-R1.2 (GND), TSV2.2 (A2); no longer J3.2
- net MOSI/SRCK: now also J3.3; no longer J3.5
- net OUT: now also EM2S1.2 (OUT), MASD-S-R1.4 (OUT), R4.1
- net ~{PON}: now also EM2S1.3 (~{PON}), MASD-S-R1.3 (~{PON})
- net ~{RESET}: now also J3.2, R13.1; no longer J3.3
- net at D5.2: now also R4.2
- net VCC renamed VBUS
Other:
- note added: "In-circuit Serial Programmer (ICSP) Bus (standard AVR layout)"
- note added: "LED-ka bude na panely."
- note added: "Nemecký modul od HKW."
- note added: "Ochrana proti opačnej polarite."
- note added: "Reichelt/MASD Napája sa cez 1V - 5V takže radšej tam dáme 3.3V"
- note removed: "Programming bus for the MCU"
- moved on the sheet: BT1, C16, C17, C5, C6, C7, C8, D2, D3, D4, D5, DCF-3850N-1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

Commit message: Zase po dlhej dobe nejaký zálohovací commit.
Other:
- note added: "Ochrana proti opačnej polarite. Samotné TSV diódy pri opačnej polarite (priepustný smer) sa chovajú ako normálne diódy (teda Uf = ~0.6V)."
- note removed: "Ochrana proti opačnej polarite."
Changed lines of the file:
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@@
 		)
 	)
-	(text "Ochrana proti opačnej polarite."
+	(text "Ochrana proti opačnej polarite.\nSamotné TSV diódy pri opačnej polarite (priepustný smer)\nsa chovajú ako normálne diódy (teda Uf = ~0.6V)."
 		(exclude_from_sim no)
 		(at 266.954 78.74 0)
@@
 			"AAAAAAAAAAAAAAAAAAAAAAAAAAAAAAAAAAAAAAAAAAAAAAAAAAAAAAAAAAAAAAAAAAAAAAAAAAAA"
 			"AAAAAAAAAAAAAAAAAAAAAAAAAAAAAAAAAAAAAAAAAAAAAAAAAAAAAAAAAAAAAAAAAAAAAAAAAAAA"
+			"AAAAAAAAAAAAAAAAAAAAAAAAAAAAAAAAAAAAAAAAAAAAAAAAAAAAAAAAAAAAAAAAAAAAAAAAAAAA"
+			"AAAAAAAAAAAAAAAAAAAAAAAAAAAAAAAAAAAAAAAAAAAAAAAAAAAAAAAAAAAAAAAAAAAAAAAAAAAA"
+			"AAAAAAAAAAAAAAAAAAAAAAAAAAAAAAAAAAAAAAAAAAAAAAAAAAAAAAAAAAAAAAAAAAAAAAAAAAAA"
+			"AAAAAAAAAAAAAAAAAAAAAAAAAAAAAAAAAAAAAAAAAAAAAAAAAAAAAAAAAAAAAAAAAAAAAAAAAAAA"
+			"AAAAAAAAAAAAAAAAAAAAAAAAAAAAAAAAAAAAAAAAAAAAAAAAAAAAAAAAAAAAAAAAAAAAAAAAAAAA"
+			"AAAAAAAAAAAAAAAAAAAAAAAAAAAAAAAAAAAAAAAAAAAAAAAAAAAAAAAAAAAAAAAAAAAAAAAAAAAA"
+			"AAAAAAAAAAAAAAAAAAAAAAAAAAAAAAAAAAAAAAAAAAAAAAAAAAAAAAAAAAAAAAAAAAAAAAAAAAAA"
+			"AAAAAAAAAAAAAAAAAAAAAAAAAAAAAAAAAAAAAAAAAAAAAAAAAAAAAAAAAAAAAAAAAAAAAAAAAAAA"
+			"AAAAAAAAAAAAAAAAAAAAAAAAAAAAAAAAAAAAAAAAAAAAAAAAAAAAAAAAAAAAAAAAAAAAAAAAAAAA"
+			"AAAAAAAAAAAAAAAAAAAAAAAAAAAAAAAAAAAAAAAAAAAAAAAAAAAAAAAAAAAAAAAAAAAAAAAAAAAA"
+			"AAAAAAAAAAAAAAAAAAAAAAAAAAAAAAAAAAAAAAAAAAAAAAAAAAAAAAAAAAAAAAAAAAAAAAAAAAAA"
+			"AAAAAAAAAAAAAAAAAAAAAAAAAAAAAAAAAAAAAAAAAAAAAAAAAAAAAAAAAAAAAAAAAAAAAAAAAAAA"
+			"AAAAAAAAAAAAAAAAAAAAAAAAAAAAAAAAAAAAAAAAAAAAAAAAAAAAAAAAAAAAAAAAAAAAAAAAAAAA"
+			"AAAAAAAAAAAAAAAAAAAAAAAAAAAAAAAAAAAAAAAAAAAAAAAAAAAAAAAAAAAAAAAAAAAAAAAAAAAA"
+			"AAAAAAAAAAAAAAAAAAAAAAAAAAAAAAAAAAAAAAAAAAAAAAAAAAAAAAAAAAAAAAAAAAAAAAAAAAAA"
+			"AAAAAAAAAAAAAAAAAAAAAAAAAAAAAAAAAAAAAAAAAAAAAAAAAAAAAAAAAAAAAAAAAAAAAAAAAAAA"
+			"AAAAAAAAAAAAAAAAAAAAAAAAAAAAAAAAAAAAAAAAAAAAAAAAAAAAAAAAAAAAAAAAAAAAAAAAAAAA"
+			"AAAAAAAAAAAAAAAAAAAAAAAAAAAAAAAAAAAAAAAAAAAAAAAAAAAAAAAAAAAAAAAAAAAAAAAAAAAA"
 			"AAAAAAAAAAAAAAAAAAAAAAAAAAAAAAAAAAAAAAAAAAAAAAAAAA=="
 		)
@@
 			"NABMADcANwBIAG0AaQBVAFMARgA1ACsAeABhAFUAQQBRAE0ANQBaAEsAdwBUAEIATQBaAGcAaQBv"
 			"AFMARAA4AHoAUAA3AFEAUABnAFAAZwA3ADAAdQA3ADkAYgBUAGsATABMAHUAZgBSAFEATwByACsA"
-			"WABBAGMAMwBSAGwAcgBsAE0AagB4AEoAQQArAHYAMABpADYAbAAzAA=="
+			"WABBAGMAMwBSAGwAcgBsAE0AagB4AEoAQQArAHYAMABpADYAbAAzADQAMwA2ADMAeABzACsAUQBP"
+			"ACsAMQBlAGQAbQA1AHIATABsAG4AQQBOAEIAYQBXADIAZQBWAFYARQBCADIAYQBvAFEAUQBVAGsA"
+			"cgBmAGMANgB1AFUAOABpAGwAZgBJAG4ATABPAE0AOAAzAGcAdwB4AGQAQgBJAGcAQQBRAFIAWgBH"
+			"ADMATgBrAEUAWQBlAHAAYwBsAE0AbABZAGIAUgA2AFEAZwBBADEAZwBHAEMAYwBjAEIASwBBAEMA"
+			"YwBGAE0AeABBADYATQBPAEYALwBzAFoAbwBOAEQAdwBkAFEANABvAE8AUgB4ADgAOQA2AC8AMwBa"
+			"AGkAUQBSAEMAQwBhAE0AdABtAEEARgBwAG0AVQBCAGgANwBKAGcAQgBvAFEAagBFADUARgBnAEMA"
+			"QwBXAC8AdgBJAEwAMgBBAGoARAAyADgAWgB6AHoAQQAwAGcAbABTAHMATQBaAEoAUQBpAGcAYQBB"
+			"AEcAMABTAGsAQQBvAHMAbgBIAFAATQB6AG8ATgBGAFoAQgBnAEMARgBoADUARQBxAFUASwBRAFkA"
+			"bQBlAGQAaQBWAFQAZwBmAHkAdQBBAHMAdgB2AFIAZwBDAHgAegBGAHQARwBmAGYAUwAxAFkAQwB5"
+			"AFoASQBJAGEATQA0AG8AbwBaADUATQA5AHEAYQAyAEEASQBTAEQAQQBaADcASwBYAFkAbABCAEkA"
+			"UwBBAEUATQA1ADUAZABLADAAbABNAG4AQQBNAGsAcQBSAHkAbgBHAFgASgBTAEkAYgBTAE8AQwBk"
+			"AEoANQBvAFgARQB4AGsASQBJAEsAQQAvAHEAQgAzAHMAZABlAEkAcgBiAEgAZABuADIAMAA4AC8A"
+			"bQBVAGsAUABYAEIAeABNAE8ASgAxAHEANAB3AGIATwBuAHYAOQBPAHkAKwBkADgAZgAvADEAbwBX"
+			"AEgAMABBAEQASgAvADEASABnADAARwBNAEEASgBBAE0AcAAwADEAMgBTAHEAVgBBAFQAcQBBAFIA"
+			"SgAvAE4AbABNAGcAbAA0AHkAaAA4AEEAdwBBAEkAWgBHADQARQBWAE8AUABEAEYARgBZADQAawBR"
+			"ADcAQgAyAGcAdgB3AG0AQQBRAHUASwBqAFEAWQBzAHcAVgBsAEEAYwB4AFoANwBDADQAWQB6AGIA"
+			"RgAwAGsASgBYAHYAbgB6AHoAbQB2AGEAaABlAHcAawBaAEEAKwBoAFIAQQBMAFkAUQBIAEIAVQBD"
+			"AEEARgB3AEQARQBDAEoAUQBCAEgARABUADMAegBBAGkAegBCAEQATwBsAEkAZwBSAEEASQBUADQA"
+			"VwB5ADIAbQBpAGYAQwBRAGIARAB5AFIAeQBHAEkAZwBaAFoAQQAyAA=="
 		)
 	)
