File: numeri-iv9-hodiny-atmega328.kicad_sch (KiCad schematic)
At the start: 55 parts, among them J1 USB_C_Receptacle_PowerOnly_6P, J2 USB-C, J3 2x3, J4 1x2, SW1 Horizontal, SW2 Vertical, U1 ATmega328-P, U2 TPIC6B595N, U3 TPIC6B595N, U4 TPIC6B595N, U5 TPIC6B595N, Y1 6MHz

Commit message: Zase po dlhej dobe nejaký zálohovací commit.
Parts:
- removed BT2: Battery_Cell, Battery:BatteryHolder_MYOUNG_BS-07-A1BJ001_CR2032, symbol Device:Battery_Cell
- removed C6: 100nF, Capacitor_THT:C_Disc_D3.0mm_W2.0mm_P2.50mm, symbol PCM_SL_Devices:Capacitor_NP
- removed D2: LED, TerminalBlock_Phoenix:TerminalBlock_Phoenix_MPT-0,5-2-2.54_1x02_P2.54mm_Horizontal, symbol PCM_SL_Devices:LED
- removed R5: 50K, PCM_SL_Devices:potentiometer_3362P, symbol Device:R_Trim
- added C1: 100nF, Capacitor_THT:C_Disc_D3.0mm_W2.0mm_P2.50mm, symbol PCM_SL_Devices:Capacitor_NP
- added C16: C_Trim, symbol Device:C_Trim
- added D2: LED_KRGB, TerminalBlock_Phoenix:TerminalBlock_Phoenix_MPT-0,5-4-2.54_1x04_P2.54mm_Horizontal, symbol Device:LED_KRGB
- added D3, D7: 1N5822, Diode_THT:D_DO-41_SOD81_P10.16mm_Horizontal, symbol Diode:1N5817
- added F2: Polyfuse, symbol Device:Polyfuse
- added J5: PINHD_1x4_Female, ExternalModules:HW_84, symbol PCM_SL_Pin_Headers:PINHD_1x4_Female
- added R14: 50K, PCM_SL_Devices:potentiometer_3362P, symbol Device:R_Trim
- added R5: 10K, Resistor_THT:R_Axial_DIN0207_L6.3mm_D2.5mm_P5.08mm_Vertical, symbol PCM_SL_Resistors:Resistor
- added SW1: Horizontal, Button_Switch_THT:SW_PUSH_6mm, symbol Switch:SW_Push
- renumbered 1m1 to 10h1, 1h1 to 10m1, 10m1 to 1h1, 10h1 to 1m1, C1 to C2, C2 to C4, C4 to C6, D3 to D4, D4 to D5, DCF-3850N-1 to DCF-3850N-1/POLLIN1, SW1 to SW2, SW2 to SW3
Connections:
- net +3.3V: now also R5.1
- net +5VREG: now also D3.1 (K), J5.2; no longer F1.2, TSV1.1 (A1), TSV2.1 (A1)
- net ADC/SCL: now also U1.28 (PC5), J5.4
- net GND: now also U2.1 (NC), U2.20 (NC_2), U3.1 (NC), U3.20 (NC_2), U4.1 (NC), U4.20 (NC_2), U5.1 (NC), U5.20 (NC_2), C1.1, D2.1 (K), J5.1, SW1.1
- net H1_2: now also 1h1.2, U4.4 (DRAIN0); no longer 10m1.2, U3.4 (DRAIN0)
- net H1_3: now also 1h1.3, U4.5 (DRAIN1); no longer 10m1.3, U3.5 (DRAIN1)
- net H1_4: now also 1h1.4, U4.6 (DRAIN2); no longer 10m1.4, U3.6 (DRAIN2)
- net H1_5: now also 1h1.5, U4.7 (DRAIN3); no longer 10m1.5, U3.7 (DRAIN3)
- net H1_6: now also 1h1.6, U4.14 (DRAIN4); no longer 10m1.6, U3.14 (DRAIN4)
- net H1_7: now also 1h1.7, U4.15 (DRAIN5); no longer 10m1.7, U3.15 (DRAIN5)
- net H1_8: now also 1h1.8, U4.16 (DRAIN6); no longer 10m1.8, U3.16 (DRAIN6)
- net H1_9: now also 1h1.9, U4.17 (DRAIN7); no longer 10m1.9, U3.17 (DRAIN7)
- net H2_2: now also 10h1.2, U5.4 (DRAIN0); no longer 1m1.2, U2.4 (DRAIN0)
- net H2_3: now also 10h1.3, U5.5 (DRAIN1); no longer 1m1.3, U2.5 (DRAIN1)
- net H2_4: now also 10h1.4, U5.6 (DRAIN2); no longer 1m1.4, U2.6 (DRAIN2)
- net H2_5: now also 10h1.5, U5.7 (DRAIN3); no longer 1m1.5, U2.7 (DRAIN3)
- net H2_6: now also 10h1.6, U5.14 (DRAIN4); no longer 1m1.6, U2.14 (DRAIN4)
- net H2_7: now also 10h1.7, U5.15 (DRAIN5); no longer 1m1.7, U2.15 (DRAIN5)
- net H2_8: now also 10h1.8, U5.16 (DRAIN6); no longer 1m1.8, U2.16 (DRAIN6)
- net H2_9: now also 10h1.9, U5.17 (DRAIN7); no longer 1m1.9, U2.17 (DRAIN7)
- net M1_2: now also 1m1.2, U2.4 (DRAIN0); no longer 10h1.2, U5.4 (DRAIN0)
- net M1_3: now also 1m1.3, U2.5 (DRAIN1); no longer 10h1.3, U5.5 (DRAIN1)
- net M1_4: now also 1m1.4, U2.6 (DRAIN2); no longer 10h1.4, U5.6 (DRAIN2)
- net M1_5: now also 1m1.5, U2.7 (DRAIN3); no longer 10h1.5, U5.7 (DRAIN3)
- net M1_6: now also 1m1.6, U2.14 (DRAIN4); no longer 10h1.6, U5.14 (DRAIN4)
- net M1_7: now also 1m1.7, U2.15 (DRAIN5); no longer 10h1.7, U5.15 (DRAIN5)
- net M1_8: now also 1m1.8, U2.16 (DRAIN6); no longer 10h1.8, U5.16 (DRAIN6)
- net M1_9: now also 1m1.9, U2.17 (DRAIN7); no longer 10h1.9, U5.17 (DRAIN7)
- net M2_2: now also 10m1.2, U3.4 (DRAIN0); no longer 1h1.2, U4.4 (DRAIN0)
- net M2_3: now also 10m1.3, U3.5 (DRAIN1); no longer 1h1.3, U4.5 (DRAIN1)
- net M2_4: now also 10m1.4, U3.6 (DRAIN2); no longer 1h1.4, U4.6 (DRAIN2)
- net M2_5: now also 10m1.5, U3.7 (DRAIN3); no longer 1h1.5, U4.7 (DRAIN3)
- net M2_6: now also 10m1.6, U3.14 (DRAIN4); no longer 1h1.6, U4.14 (DRAIN4)
- net M2_7: now also 10m1.7, U3.15 (DRAIN5); no longer 1h1.7, U4.15 (DRAIN5)
- net M2_8: now also 10m1.8, U3.16 (DRAIN6); no longer 1h1.8, U4.16 (DRAIN6)
- net M2_9: now also 10m1.9, U3.17 (DRAIN7); no longer 1h1.9, U4.17 (DRAIN7)
- net MISO/HBTN: now also U1.5 ((PWM)PD3)
- net MOSI/SRCK: now also U1.14 (PB0); no longer U1.4 (PD2)
- net OUT: now also U1.26 (PC3)
- net RCK: now also U1.13 (PD7); no longer U1.6 (PD4)
- net SER_IN: now also U1.15 (PB1)
- net VBTN: now also U1.4 (PD2)
- net ~{G}~: now also U1.12 ((PWM)PD6); no longer U1.5 ((PWM)PD3)
- net ~{PON}: now also D7.2 (A), R5.2
- net ~{RESET}: now also SW1.2
- net LED_R: now reaches U1.17 ((PWM)PB3)
- net LED_R: now also D2.2 (RA)
- net LED_G: now reaches U1.18 ((PWM)PB4)
- net LED_G: now also D2.3 (GA)
- net LED_B: now reaches U1.19 ((PWM)PB5)
- net LED_B: now also D2.4 (BA)
- net at U1.21 (AREF): now also C1.2
- net SDA: now reaches U1.27 (PC4)
- net SDA: now also J5.3
- net at D5.2 (A): now also F2.1; no longer BT1.1 (+)
- new net: D7.1 (K), U1.6 (PD4)
- new net: BT1.1 (+), F2.2
- new net: R14.1, R14.2
- new net: D3.2 (A), F1.2, TSV1.1 (A1), TSV2.1 (A1)
Other:
- note added: "Ochrana pred HIGH stavom pinu. Dioda povoluje len LOW stav."
- note added: "Ochrana proti opačnej polarite. Samotné TSV diódy pri opačnej polarite (priepustný smer) sa chovajú ako normálne diódy (teda Uf = ~0.6V)."
- note added: "Podľa datasheetu majú byť C2 a C4 rovnaké."
- note added: "Podľa datasheetu piny NC nemajú žiadne interné prepojenie v čipe a mali by byť pripojené ku GND pre lepšiu distribúciu tepla."
- note added: "Pull-up rezistor"
- note added: "RTC Module"
- note added: "Sofvérovo kontrolované indikačná RGB LED-ka pre DCF77 modul. Všetky farby by mali byť cez PWM."
- note added: "TODO: Treba dopočítať rezistory. TODO: Trimmer implementovať softvérovo."
- note removed: "Ochrana proti opačnej polarite."
- moved on the sheet: 10h1, 10m1, 1h1, 1m1, BT1, C11, C12, C14, C15, C2, C4, C6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

Commit message: preventivne
Parts:
- removed BT1: CR2032, Battery:BatteryHolder_Keystone_CR2032_Vertical, symbol Device:Battery_Cell
- removed C10, C6: 100nF, Capacitor_THT:C_Disc_D3.0mm_W2.0mm_P2.50mm, symbol PCM_SL_Devices:Capacitor_NP
- removed C13: 3,3uF, Capacitor_THT:CP_Radial_D5.0mm_P2.00mm, symbol PCM_SL_Capacitors:100uF_10V
- removed C16: C_Trim, symbol Device:C_Trim
- removed C3: 10uF, Capacitor_THT:CP_Radial_D5.0mm_P2.00mm, symbol PCM_SL_Capacitors:10uF_16V
- removed C9: 4.7uF, Capacitor_THT:CP_Radial_D5.0mm_P2.00mm, symbol PCM_SL_Capacitors:4.7uF_16V
- removed D4, D5, D7: 1N5822, Diode_THT:D_DO-41_SOD81_P10.16mm_Horizontal, symbol Diode:1N5817
- removed DCF-3850N-1/POLLIN1, EM2S1, MASD-S-R1: DCF77, Connector_PinSocket_2.54mm:PinSocket_1x04_P2.54mm_Vertical, symbol DCF77_Module_DCF-3850N-1:con-amp-quick_125_M04
- removed F2: Polyfuse, symbol Device:Polyfuse
- removed J5: PINHD_1x4_Female, ExternalModules:HW_84, symbol PCM_SL_Pin_Headers:PINHD_1x4_Female
- removed R6: 10K, Resistor_THT:R_Axial_DIN0207_L6.3mm_D2.5mm_P5.08mm_Vertical, symbol PCM_SL_Resistors:Resistor
- added C15, C16: 4.7uF, Capacitor_THT:C_Disc_D4.3mm_W1.9mm_P5.00mm, symbol PCM_SL_Devices:Capacitor_NP
- added C4, C5: 100nF, Capacitor_THT:C_Disc_D3.0mm_W2.0mm_P2.50mm, symbol PCM_SL_Devices:Capacitor_NP
- added D2: 1N5822, Diode_THT:D_DO-41_SOD81_P10.16mm_Horizontal, symbol Diode:1N5817
- added DCF77-MODUL1: DCF77, Connector_PinSocket_2.54mm:PinSocket_1x04_P2.54mm_Vertical, symbol DCF77_Module_DCF-3850N-1:con-amp-quick_125_M04
- added J4: Screw_Terminal_01x04, symbol Connector:Screw_Terminal_01x04
- added J7: 1x2, Connector_PinHeader_2.54mm:PinHeader_1x02_P2.54mm_Vertical, symbol PCM_SL_Pin_Headers:PINHD_1x2_Male
- added J8: DS3231, ExternalModules:HW_84, symbol PCM_SL_Pin_Headers:PINHD_1x4_Female
- added R13: 1R±5%, Resistor_THT:R_Axial_DIN0414_L11.9mm_D4.5mm_P15.24mm_Horizontal, symbol PCM_SL_Resistors:Resistor
- C1: renamed from C2; DType (none) -> C0G/NP0
- C2: renamed from C4; DType (none) -> C0G/NP0
- C8: renamed from C5; value 100nF -> 1uF; U 50V -> 25V
- SW1: Typ Control -> RESET
- TSV1, TSV2: footprint Diode_THT:D_DO-201AE_P15.24mm_Horizontal -> Diode_THT:D_DO-15_P12.70mm_Horizontal
- U1: footprint Package_DIP:DIP-28_W7.62mm -> Package_DIP:DIP-28_W7.62mm_Socket
- renumbered C14 to C13, C15 to C14, C1 to C3, C7 to C6, C8 to C7, D2 to D1, D1 to D3, D3 to D4, J3 to J2, J1 to J3, J2 to J5, J4 to J6, R3 to R2, R4 to R3, R14 to R4, R2 to R6
Connections:
- net +3.3V: now also R5.2; no longer R5.1
- net +5VBAT: no longer R1.2, U1.20 (AVCC), U1.7 (VCC)
- net +5VREG: no longer D4.1 (K), R8.2
- net ADC/SCL: now also J8.4
- net GND: now also C15.1, C16.1, C4.1, C5.2, J8.1
- net RX: now also J7.2
- net SDA: now also J8.3
- net TX: now also J7.1
- net ~{PON}: now also R5.1, D2.2 (A); no longer R5.2
- net at U1.21 (AREF): now also C5.1; no longer C3.2
- net at U1.25 (PC2): now also R4.2
- net PD4: now reaches U1.6 (PD4)
- net PD4: now also D2.1 (K)
- net +5V: now reaches R4.1
- net +5V: now also C3.2, D4.1 (K), R1.2, R8.2, U1.20 (AVCC), U1.7 (VCC), C15.2, C16.2, C4.2, J8.2; no longer R4.2
- new net: DCF77-MODUL1.4, J4.1 (Pin_1)
- new net: DCF77-MODUL1.3, J4.2 (Pin_2)
- new net: DCF77-MODUL1.2, J4.3 (Pin_3)
- new net: DCF77-MODUL1.2, J4.4 (Pin_4)
Other:
- note added: "Indikátor synchronizácie"
- note added: "Keďže existuje veľa roznych verzií modulov pre príjimanie signálu DCF77 a väčšina sa lýši len poradím pinov prípadne veľkosťou napájacieho napätia (3.3V/5V), potrebujeme flexibilné zapojenie, ktoré bude podporovať všetky tieto moduly. V našom prípade to riešime cez 4-pinovú svorkovnicu, ktorej káble sa dajú poprehadzovať podľa potreby."
- note added: "Piny PON a OUT vieme zmeniť v softvéri."
- note added: "Podľa datasheetu majú byť C2 a C4 rovnaké. Pod kryštáľom nemajú byť žiadne iné spoje ani liata meď."
- note added: "Pojistka môže byť montovaná aj na krabičke. Nemalo by byť treba ju meniť, takže to asi nie je treba."
- note added: "Pull-up rezistor zaistí východzí 3.3V HIGH stav."
- note added: "RGB LED-ka bude na panely."
- note added: "RTC"
- note added: "Schottkyho dióda zábrani 5V HIGH stavu z MCU aby poškodil 3.3V modul, v prípade chyby v sofvéri."
- note added: "Upravovanie max. jasu RGB diódy."
- note removed: "Battery backup"
- note removed: "Detekcia napájania"
- note removed: "LED-ka bude na panely."
- note removed: "Nemecký modul od HKW."
- note removed: "Podľa datasheetu majú byť C2 a C4 rovnaké."
- note removed: "Pull-up rezistor"
- note removed: "RTC Module"
- note removed: "Reichelt/MASD Napája sa cez 1V - 5V takže radšej tam dáme 3.3V"
- note removed: "The fuse can be on the case as well."
- note removed: "~ marks a PWM pin"
- moved on the sheet: C1, C2, C3, C8, D1, D3, J2, J6, R1, R4, R6, SW1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

Commit message: preventivne
Parts:
- removed D3: 1N4728, Diode_THT:D_DO-41_SOD81_P10.16mm_Horizontal, symbol Diode:1N47xxA
- removed D4: 1N5822, Diode_THT:D_DO-41_SOD81_P10.16mm_Horizontal, symbol Diode:1N5817
- removed J7: 1x2, Connector_PinHeader_2.54mm:PinHeader_1x02_P2.54mm_Vertical, symbol PCM_SL_Pin_Headers:PINHD_1x2_Male
- removed R4: 50K, PCM_SL_Devices:potentiometer_3362P, symbol Device:R_Trim
- removed R6: 2K5, Resistor_THT:R_Axial_DIN0207_L6.3mm_D2.5mm_P10.16mm_Horizontal, symbol PCM_SL_Resistors:Resistor
- added C15, C9: 1uF, Capacitor_THT:C_Disc_D3.0mm_W2.0mm_P2.50mm, symbol PCM_SL_Devices:Capacitor_NP
- added D2: 1N4728, Diode_THT:D_DO-41_SOD81_P10.16mm_Horizontal, symbol Diode:1N47xxA
- added FB1: 79R@100MHz, symbol Device:FerriteBead
- added J4: PINHD_1x3_Female, Connector_PinSocket_2.54mm:PinSocket_1x03_P2.54mm_Vertical, symbol PCM_SL_Pin_Headers:PINHD_1x3_Female
- added Q1, Q2: BC557, Package_TO_SOT_THT:TO-92_Inline, symbol Transistor_BJT:BC557
- added R13: 10R, Resistor_THT:R_Axial_DIN0207_L6.3mm_D2.5mm_P10.16mm_Horizontal, symbol PCM_SL_Resistors:Resistor
- added R14: 330R, Resistor_THT:R_Axial_DIN0207_L6.3mm_D2.5mm_P10.16mm_Horizontal, symbol PCM_SL_Resistors:Resistor
- added R16: 20R, Resistor_THT:R_Axial_DIN0207_L6.3mm_D2.5mm_P10.16mm_Horizontal, symbol PCM_SL_Resistors:Resistor
- added R17: 550R, Resistor_THT:R_Axial_DIN0207_L6.3mm_D2.5mm_P10.16mm_Horizontal, symbol PCM_SL_Resistors:Resistor
- added RV1, RV2: 50K, PCM_SL_Devices:potentiometer_3362P, symbol Device:R_Potentiometer_Trim
- C1, C2: value 12.5pF -> 12p5
- C10: renamed from C15; value 4.7uF -> 4u7
- C11: renamed from C16; value 4.7uF -> 4u7
- C8: value 1uF -> 10nF; U 25V -> 50V
- F1: value F1.25A -> F1A25
- J5: renamed from J8; value DS3231 -> HW-084
- R1: footprint Resistor_THT:R_Axial_DIN0207_L6.3mm_D2.5mm_P5.08mm_Vertical -> Resistor_THT:R_Axial_DIN0207_L6.3mm_D2.5mm_P10.16mm_Horizontal
- R6: renamed from R7; footprint Resistor_THT:R_Axial_DIN0207_L6.3mm_D2.5mm_P5.08mm_Vertical -> Resistor_THT:R_Axial_DIN0207_L6.3mm_D2.5mm_P10.16mm_Horizontal
- RGB_LED1: renamed from D1; value LED_KRGB -> RGB_LED
- SW1: value Horizontal -> RESET; Typ RESET -> (none)
- TSV1: Voltage 5.8V -> 5V8
- TSV2: value BZW06-5V8 -> 1N5908; Voltage 5.8V -> 5V
- renumbered C11 to C12, C12 to C13, C13 to C14, C14 to C16, D2 to D1, J2 to ICSP1, J3 to J1, J4 to J2, J5 to J3, R13 to R15, R9 to R7, R10 to R9, J6 to SERIAL1
Connections:
- net +5VBAT is gone; now on net +5V: ICSP1.5, R6.2
- net +3.3V: now also J4.1; no longer C8.2, R5.2
- net +5V: now also R11.2, R12.2, R15.2, R7.2, R9.2, C9.2, FB1.2, J4.3, R13.2, RV1.3, RV2.1
- net GND: now also SW2.1, C15.1, C9.1, D2.2 (A), R14.1, R17.1, RV1.1, RV2.3; no longer SW2.2
- net MISO/HBTN: now also SW2.2; no longer SW2.1
- net PB2: now reaches U1.16 (PB2)
- net PB2: now also D1.1 (K)
- net at U1.23 (PC0): now also RV1.2
- net DEC_OUT: now reaches U1.25 (PC2)
- net DEC_OUT: now also Q2.1 (C), R17.2
- net +5V_DEC: now reaches R15.1
- net +5V_DEC: now also 10h1.1, 10m1.1, 1h1.1, 1m1.1, C12.2, C13.2, C14.2, C16.2, U2.2 (VCC), U3.2 (VCC), U4.2 (VCC), U5.2 (VCC), R16.2
- net at F1.2, TSV1.1 (A1), TSV2.1 (A1): now also C8.2, FB1.1
- removed net +5VREG: 10h1.1, 10m1.1, 1h1.1, 1m1.1, C12.2, C13.2, C14.2, C16.2, R11.2, R12.2, R7.2, R9.2, U2.2 (VCC), U3.2 (VCC), U4.2 (VCC), U5.2 (VCC)
- net ADC/SCL renamed SCL
- net PD4: no longer names the net of U1.6 (PD4)
- net PD4: no longer D1.1 (K)
- new net: Q1.1 (C), Q1.2 (B), Q2.2 (B), R14.2
- new net: Q2.3 (E), R16.1
- new net: Q1.3 (E), R13.1
- new net +3V3: C15.2, D2.1 (K), RV2.2
- new net +5V/+3V3: J4.2, R5.2
Other:
- note added: "Keďže existuje veľa roznych verzií modulov pre príjimanie signálu DCF77 a väčšina sa lýši len poradím pinov prípadne veľkosťou napájacieho napätia (3V3/5V), potrebujeme flexibilné zapojenie, ktoré bude podporovať všetky tieto moduly. V našom prípade to riešime cez 4-pinovú svorkovnicu, ktorej káble sa dajú poprehadzovať podľa potreby."
- note added: "Modul zapojenia DS3231 SMD čipu so zabudovanou batériou. Chybovosť čipu okolo ~2ppm prvých 5 rokov, takže max. odchylka ~60 s za rok."
- note added: "Napájanie a ovládanie modulu príjimača"
- note added: "Napätie: R: 2V-2V2 G/B: 3V-3V2"
- note added: "Príjimač signálu atomových hodín"
- note added: "RG = RB = (5V-2V)/8*10^3A = 375R RR = (5V-3V)/8*10^3A = 250R"
- note added: "Regulácia prúdu pomocou trimra podľa potreby pripojených záťaží."
- note added: "Schottkyho dióda zábrani 5V HIGH stavu z MCU aby poškodil 3V3 modul, v prípade chyby v sofvéri."
- note added: "Senzor prúdového odberu displeja"
- note added: "TODO: Treba dopočítať rezistory."
- note added: "Voľba medzi +5V a +3V3 pomocou mostíkovej prepojky."
- note added: "Zapojenie modulu príjimača"
- note added: "Zdroj Napätia 3V3"
- note removed: "Atomic clock signal receiver"
- note removed: "Keďže existuje veľa roznych verzií modulov pre príjimanie signálu DCF77 a väčšina sa lýši len poradím pinov prípadne veľkosťou napájacieho napätia (3.3V/5V), potrebujeme flexibilné zapojenie, ktoré bude podporovať všetky tieto moduly. V našom prípade to riešime cez 4-pinovú svorkovnicu, ktorej káble sa dajú poprehadzovať podľa potreby."
- note removed: "Ochrana pred HIGH stavom pinu. Dioda povoluje len LOW stav."
- note removed: "R = 5V/2mA = 2K5"
- note removed: "Schottkyho dióda zábrani 5V HIGH stavu z MCU aby poškodil 3.3V modul, v prípade chyby v sofvéri."
- note removed: "TODO: Treba dopočítať rezistory. TODO: Trimmer implementovať softvérovo."
- company: (none) -> Filip Mitka
- title: Numitron Clock with DCF77 -> Numeri - Rádiovo riadené numitronové hodiny
- moved on the sheet: C10, C11, C6, D1, DCF77-MODUL1, F1, ICSP1, J2, J5, R15, R5, R8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

Commit message: preventivne
Parts:
- FB1: footprint (none) -> Inductor_THT:L_Axial_L5.0mm_D3.6mm_P10.00mm_Horizontal_Murata_BL01RN1A2A2
- J2: footprint (none) -> TerminalBlock_Phoenix:TerminalBlock_Phoenix_MPT-0,5-4-2.54_1x04_P2.54mm_Horizontal
Connections:
- net at J2.4 (Pin_4): now also DCF77-MODUL1.1; no longer DCF77-MODUL1.2
Changed lines of the file:
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@@
 	(text "Ochrana proti opačnej polarite.\nSamotné TSV diódy pri opačnej polarite (priepustný smer)\nsa chovajú ako normálne diódy (teda Uf = ~0.6V)."
 		(exclude_from_sim no)
-		(at 273.558 57.912 0)
+		(at 275.59 57.15 0)
 		(effects
 			(font
@@
 			"AAAAAAAAAAAAAAAAAAAAAAAAAAAAAAAAAAAAAAAAAAAAAAAAAAAAAAAAAAAAAAAAAAAAAAAAAAAA"
 			"AAAAAAAAAAAAAAAAAAAAAAAAAAAAAAAAAAAAAAAAAAAAAAAAAAAAAAAAAAAAAAAAAAAAAAAAAAAA"
+			"AAAAAAAAAAAAAAAAAAAAAAAAAAAAAAAAAAAAAAAAAAAAAAAAAAAAAAAAAAAAAAAAAAAAAAAAAAAA"
+			"AAAAAAAAAAAAAAAAAAAAAAAAAAAAAAAAAAAAAAAAAAAAAAAAAAAAAAAAAAAAAAAAAAAAAAAAAAAA"
+			"AAAAAAAAAAAAAAAAAAAAAAAAAAAAAAAAAAAAAAAAAAAAAAAAAAAAAAAAAAAAAAAAAAAAAAAAAAAA"
+			"AAAAAAAAAAAAAAAAAAAAAAAAAAAAAAAAAAAAAAAAAAAAAAAAAAAAAAAAAAAAAAAAAAAAAAAAAAAA"
+			"AAAAAAAAAAAAAAAAAAAAAAAAAAAAAAAAAAAAAAAAAAAAAAAAAAAAAAAAAAAAAAAAAAAAAAAAAAAA"
+			"AAAAAAAAAAAAAAAAAAAAAAAAAAAAAAAAAAAAAAAAAAAAAAAAAAAAAAAAAAAAAAAAAAAAAAAAAAAA"
+			"AAAAAAAAAAAAAAAAAAAAAAAAAAAAAAAAAAAAAAAAAAAAAAAAAAAAAAAAAAAAAAAAAAAAAAAAAAAA"
+			"AAAAAAAAAAAAAAAAAAAAAAAAAAAAAAAAAAAAAAAAAAAAAAAAAAAAAAAAAAAAAAAAAAAAAAAAAAAA"
+			"AAAAAAAAAAAAAAAAAAAAAAAAAAAAAAAAAAAAAAAAAAAAAAAAAAAAAAAAAAAAAAAAAAAAAAAAAAAA"
+			"AAAAAAAAAAAAAAAAAAAAAAAAAAAAAAAAAAAAAAAAAAAAAAAAAAAAAAAAAAAAAAAAAAAAAAAAAAAA"
+			"AAAAAAAAAAAAAAAAAAAAAAAAAAAAAAAAAAAAAAAAAAAAAAAAAAAAAAAAAAAAAAAAAAAAAAAAAAAA"
+			"AAAAAAAAAAAAAAAAAAAAAAAAAAAAAAAAAAAAAAAAAAAAAAAAAAAAAAAAAAAAAAAAAAAAAAAAAAAA"
+			"AAAAAAAAAAAAAAAAAAAAAAAAAAAAAAAAAAAAAAAAAAAAAAAAAAAAAAAAAAAAAAAAAAAAAAAAAAAA"
+			"AAAAAAAAAAAAAAAAAAAAAAAAAAAAAAAAAAAAAAAAAAAAAAAAAAAAAAAAAAAAAAAAAAAAAAAAAAAA"
+			"AAAAAAAAAAAAAAAAAAAAAAAAAAAAAAAAAAAAAAAAAAAAAAAAAAAAAAAAAAAAAAAAAAAAAAAAAAAA"
+			"AAAAAAAAAAAAAAAAAAAAAAAAAAAAAAAAAAAAAAAAAAAAAAAAAAAAAAAAAAAAAAAAAAAAAAAAAAAA"
+			"AAAAAAAAAAAAAAAAAAAAAAAAAAAAAAAAAAAAAAAAAAAAAAAAAAAAAAAAAAAAAAAAAAAAAAAAAAAA"
+			"AAAAAAAAAAAAAAAAAAAAAAAAAAAAAAAAAAAAAAAAAAAAAAAAAAAAAAAAAAAAAAAAAAAAAAAAAAAA"
 			"AAAAAAAAAAAAAAAAAAAAAAAAAAAAAAAAAAAAAAAAAAAAAAAAAAAAAA=="
 		)
@@
 			"NQBsAGIAYwArAHIATQA3AGYAbgB6ADUARQBsAFEAVABvAFUAUQA1AFAAdgBvAFAALwBnAEIAVwBB"
 			"AEIATABsADYAUABpAFAAdgBQAGYAcQBGADcALwBXAGIAcgArAHYARgBsAFQAOQBtAGQAawBiAFgA"
-			"MwB1AG0ARQBUAFIAZwBaAGIARgBqADUAKwBLADQAcwBqAFgATAB0ADYANgBzAA=="
+			"MwB1AG0ARQBUAFIAZwBaAGIARgBqADUAKwBLADQAcwBqAFgATAB0ADYANgBzADIAcAByAEwASwBq"
+			"AEwAdABRAHMAYgBLADgAdAB3AFIAWQBmAE4AVABZAFYAaABMAFIAcABMADIAcgBCAGEAZQB0AHIA"
+			"RwBaAFIAWABjADcAaQBoAEsAbQBFAGcAUQBGAHQAbQArADUALwBPAFcAdgBPAHAARABpAHMAaQBn"
+			"AEIAUQBaAEwANwBRAFgAawBjAEEAOABOAFEAYgBkAHkAMwAwAFMAdQBhAHQAWgBKAHYAbQB1ADIA"
+			"MAAwAFUAUgBpAFkAQQBCAEYAQwBFAG8ARABjAFcAMgBKAGoAZABvADcAcAA1AGYARQB1AGwAbAB2"
+			"AHAANABPAEwAWgAyAFUAawA0AHkAbgBmAGMASgBUAG4ASwB1ACsATQBwAHYAeQBUAFMANwA3AHcA"
+			"MQBHAGUAZABCAHIALwBrAGUAVwAzAGsAcwArAG4AZgBmACsAWABlAGkANwArAHgATgBpADMANwBX"
+			"AHEAVgB4AE4ASwBWAE0ARgBuAHUAeABLAEkAWQA3AEUAeABWAE8AawA4AGwAVQA1AFAAVgByAFgA"
+			"dgBiAGkAcAAzADMAeABxAHgAaQB1AHcAaQBkAFkARQBiAFEANgBYAGkAcwBQAC8AVwBwAFEAVwBE"
+			"AFMANgBnAEkAVgBOAFEAQgA2AGkAQQBkAEgAVQBZAFEAYgBQAEkAdwBnAHQAMAB3AHcAZABZAE0A"
+			"MABSADAAZABwADEATgBsADEAZgAzAHoAVQBaAEkAZwB3AGcATgBlAEsASgB4AE0AOABIAEIAbQBm"
+			"AEgAaABtAHUAbgByAEQAVgBxAFEAYwBzAEkAeAAzAEcAYwBoADMARABaADEAMwBIADIAVwA3ADAA"
+			"LwA3AHkAYQBGAHoAQwBIAE4AUABkACsANwA2AHMAQgA0AFgARABUAHoAVQBtADMAawBxAE4AUABQ"
+			"AFEARwBVAEEAWQBYAGYAcABLAFUAKwA1AC8ANAByADEAYQBIAFMAcAAwAFcAcgBjAGUAZQArAFMA"
+			"QgA2AFoAUgBHAGQAYQBpAEYAWABpAGgAZwBMAEoANwBwAG4AUABEADMAQQBYAHUATgBhAHUAYQB1"
+			"AHoAcgAvADUAWABIAHYAawBLAHIAZQBmAHcAegBOAFYARgBoAFAASwBRAE4AdgBXADYAYwA0ADUA"
+			"WgB6AFgANABYAGwAUAB4AGQAMQAzADMAUAAzADIAZAA4AHQAVwBCAHUAYgBSAHkAdQBBAHMAaABh"
+			"AFkAYwBuAGYAeQB4ADgAMwBEAHMAbwBmAHoAeAB0ADYAKwAvADcAQQBjAFYAawArAGYATgB1AG0A"
+			"MwBuADIAVwAxADMAQgBNAGMAZABEAHEAKwBGAFQAdgBPAGEAUwB5ADUAZQByAA=="
 		)
 	)
@@
 			)
 		)
-		(property "Footprint" ""
+		(property "Footprint" "TerminalBlock_Phoenix:TerminalBlock_Phoenix_MPT-0,5-4-2.54_1x04_P2.54mm_Horizontal"
 			(at 100.33 340.36 0)
 			(effects
@@
 			)
 		)
-		(property "Footprint" ""
+		(property "Footprint" "Inductor_THT:L_Axial_L5.0mm_D3.6mm_P10.00mm_Horizontal_Murata_BL01RN1A2A2"
 			(at 265.43 70.358 90)
 			(effects
@@
 		(pin "4"
 		)
-		(pin "2"
+		(pin "1"
 		)
 		(instances

Commit message: preventívne
Parts:
- removed R17: 550R, Resistor_THT:R_Axial_DIN0207_L6.3mm_D2.5mm_P10.16mm_Horizontal, symbol PCM_SL_Resistors:Resistor
- added R4: 1K, Potentiometer_THT:Potentiometer_Bourns_3296W_Vertical, symbol Device:R_Trim
- C12, C13, C14, C16, C3, C4, C5, C6, C7: footprint Capacitor_THT:C_Disc_D3.0mm_W2.0mm_P2.50mm -> Capacitor_THT:C_Disc_D6.0mm_W2.5mm_P5.00mm
- J4: footprint Connector_PinSocket_2.54mm:PinSocket_1x03_P2.54mm_Vertical -> Connector_PinHeader_2.54mm:PinHeader_1x03_P2.54mm_Vertical
- R1, R13, R16: footprint Resistor_THT:R_Axial_DIN0207_L6.3mm_D2.5mm_P10.16mm_Horizontal -> Resistor_THT:R_Axial_DIN0207_L6.3mm_D2.5mm_P5.08mm_Vertical
- R11, R12, R6, R7, R9: footprint Resistor_THT:R_Axial_DIN0207_L6.3mm_D2.5mm_P10.16mm_Horizontal -> Resistor_THT:R_Axial_DIN0207_L6.3mm_D2.5mm_P15.24mm_Horizontal
- R15: footprint Resistor_THT:R_Axial_DIN0414_L11.9mm_D4.5mm_P15.24mm_Horizontal -> Resistor_THT:R_Axial_DIN0414_L11.9mm_D4.5mm_P25.40mm_Horizontal
- R8: footprint Resistor_THT:R_Axial_DIN0207_L6.3mm_D2.5mm_P2.54mm_Vertical -> Resistor_THT:R_Axial_DIN0207_L6.3mm_D2.5mm_P10.16mm_Horizontal
- SERIAL1: footprint Connector_PinHeader_2.54mm:PinHeader_1x02_P2.54mm_Vertical -> Connector_PinSocket_2.54mm:PinSocket_1x02_P2.54mm_Vertical
- SW2, SW3: footprint TerminalBlock_Phoenix:TerminalBlock_Phoenix_MPT-0,5-2-2.54_1x02_P2.54mm_Horizontal -> TerminalBlock_Phoenix:TerminalBlock_Phoenix_MPT-0,5-2-2.54_1x02_P2.54mm_Horizontal_RAW
- U2, U3, U4, U5: footprint Package_DIP:DIP-20_W7.62mm_Socket -> Package_DIP:DIP-20_W7.62mm_Socket_With_IC
Connections:
- net +3.3V is gone; now on net +3V3: J4.1
- net DEC_OUT: now also R4.1
- net GND: now also R4.2
