File: numeri-iv9-hodiny-atmega328.kicad_sch (KiCad schematic)
At the start: 63 parts, among them J1 USB_C_Receptacle_PowerOnly_6P, J2 Screw_Terminal_01x04, J3 USB-C, J4 PINHD_1x3_Female, J5 HW-084, Q1 BC557, Q2 BC557, SW1 RESET, SW2 Horizontal, SW3 Vertical, U1 ATmega328-P, U2 TPIC6B595N, U3 TPIC6B595N, U4 TPIC6B595N, U5 TPIC6B595N, Y1 6MHz

Commit message: preventívne
Parts:
- added R10: 619R, Resistor_THT:R_Axial_DIN0207_L6.3mm_D2.5mm_P7.62mm_Horizontal, symbol PCM_SL_Resistors:Resistor
- added R17: 464R, Resistor_THT:R_Axial_DIN0207_L6.3mm_D2.5mm_P2.54mm_Vertical, symbol PCM_SL_Resistors:Resistor
- added R18: 464R, Resistor_THT:R_Axial_DIN0207_L6.3mm_D2.5mm_P7.62mm_Horizontal, symbol PCM_SL_Resistors:Resistor
- added R19: 330R, Resistor_THT:R_Axial_DIN0207_L6.3mm_D2.5mm_P7.62mm_Horizontal, symbol PCM_SL_Resistors:Resistor
- C1, C2: value 12p5 -> 33pF±5%
- R16: footprint Resistor_THT:R_Axial_DIN0207_L6.3mm_D2.5mm_P5.08mm_Vertical -> Resistor_THT:R_Axial_DIN0207_L6.3mm_D2.5mm_P10.16mm_Horizontal
- Y1: value 6MHz -> 16MHz±20ppm
Connections:
- net LED_B: now also R18.2; no longer RGB_LED1.4 (BA)
- net LED_G: now also R17.2; no longer RGB_LED1.3 (GA)
- net LED_R: now also R10.2; no longer RGB_LED1.2 (RA)
- new net: R10.1, RGB_LED1.2 (RA)
- new net: R17.1, RGB_LED1.3 (GA)
- new net: R18.1, RGB_LED1.4 (BA)
Other:
- note added: "CL = (C1 * C2) / (C1 + C2) + Cstray C1 = C2 = 2CL + 2Cstray pre CL = 30pF; Cstray = 5pF => C1 = C2 = 70pF"
- note added: "Napätie (podľa meraní): R: 1V72 - 1V92 G/B: 2V48 - 3V Maximálny prúd pre farbu: 5mA"
- note added: "RG = RB = (5V-2V48)/5*10^-3A = 544 (464) RR = (5V-1V72)/5*10^-3A = 656 (619) * Zaokrúhlene na najbližšiu bežnú hodnotu."
- note added: "Softvérovo kontrolované indikačná RGB LED-ka pre DCF77 modul. Všetky farby by mali byť cez PWM."
- note removed: "Napätie: R: 2V-2V2 G/B: 3V-3V2"
- note removed: "RG = RB = (5V-2V)/8*10^3A = 375R RR = (5V-3V)/8*10^3A = 250R"
- note removed: "Sofvérovo kontrolované indikačná RGB LED-ka pre DCF77 modul. Všetky farby by mali byť cez PWM."
- note removed: "TODO: Treba dopočítať rezistory."
- moved on the sheet: RGB_LED1

Commit message: Pridaná bloková schéma.
Parts:
- removed 10h1, 10m1, 1h1, 1m1: IV-9, VacuumTubes:IV-9_External_Socket_Asymetric, symbol VacuumTubes:IV-9
- removed C1, C2: 33pF±5%, Capacitor_THT:C_Disc_D3.0mm_W2.0mm_P2.50mm, symbol PCM_SL_Devices:Capacitor_NP
- removed C10, C11: 4u7, Capacitor_THT:C_Disc_D4.3mm_W1.9mm_P5.00mm, symbol PCM_SL_Devices:Capacitor_NP
- removed C12, C13, C14, C16, C3, C4, C5, C6, C7: 100nF, Capacitor_THT:C_Disc_D6.0mm_W2.5mm_P5.00mm, symbol PCM_SL_Devices:Capacitor_NP
- removed C15, C9: 1uF, Capacitor_THT:C_Disc_D3.0mm_W2.0mm_P2.50mm, symbol PCM_SL_Devices:Capacitor_NP
- removed C8: 10nF, Capacitor_THT:C_Disc_D3.0mm_W2.0mm_P2.50mm, symbol PCM_SL_Devices:Capacitor_NP
- removed D1: 1N5822, Diode_THT:D_DO-41_SOD81_P10.16mm_Horizontal, symbol Diode:1N5817
- removed D2: 1N4728, Diode_THT:D_DO-41_SOD81_P10.16mm_Horizontal, symbol Diode:1N47xxA
- removed DCF77-MODUL1: DCF77, Connector_PinSocket_2.54mm:PinSocket_1x04_P2.54mm_Vertical, symbol DCF77_Module_DCF-3850N-1:con-amp-quick_125_M04
- removed F1: F1A25, Fuse:Fuseholder_Cylinder-5x20mm_Schurter_0031_8201_Horizontal_Open, symbol Device:Fuse
- removed FB1: 79R@100MHz, Inductor_THT:L_Axial_L5.0mm_D3.6mm_P10.00mm_Horizontal_Murata_BL01RN1A2A2, symbol Device:FerriteBead
- removed ICSP1: 2x3, Connector_PinHeader_2.54mm:PinHeader_2x03_P2.54mm_Vertical, symbol PCM_SL_Pin_Headers:PINHD_2x3_Male
- removed J1: USB_C_Receptacle_PowerOnly_6P, symbol Connector:USB_C_Receptacle_PowerOnly_6P
- removed J2: Screw_Terminal_01x04, TerminalBlock_Phoenix:TerminalBlock_Phoenix_MPT-0,5-4-2.54_1x04_P2.54mm_Horizontal, symbol Connector:Screw_Terminal_01x04
- removed J3: USB-C, TerminalBlock_Phoenix:TerminalBlock_Phoenix_PT-1,5-2-5.0-H_1x02_P5.00mm_Horizontal, symbol PCM_SL_Screw_Terminal:Screw_Terminal_2_P3.50mm
- removed J4: PINHD_1x3_Female, Connector_PinHeader_2.54mm:PinHeader_1x03_P2.54mm_Vertical, symbol PCM_SL_Pin_Headers:PINHD_1x3_Female
- removed J5: HW-084, ExternalModules:HW_84, symbol PCM_SL_Pin_Headers:PINHD_1x4_Female
- removed Q1, Q2: BC557, Package_TO_SOT_THT:TO-92_Inline, symbol Transistor_BJT:BC557
- removed R1, R5: 10K, Resistor_THT:R_Axial_DIN0207_L6.3mm_D2.5mm_P5.08mm_Vertical, symbol PCM_SL_Resistors:Resistor
- removed R10: 619R, Resistor_THT:R_Axial_DIN0207_L6.3mm_D2.5mm_P7.62mm_Horizontal, symbol PCM_SL_Resistors:Resistor
- removed R11, R12, R6, R7, R9: 10K, Resistor_THT:R_Axial_DIN0207_L6.3mm_D2.5mm_P15.24mm_Horizontal, symbol PCM_SL_Resistors:Resistor
- removed R13: 10R, Resistor_THT:R_Axial_DIN0207_L6.3mm_D2.5mm_P5.08mm_Vertical, symbol PCM_SL_Resistors:Resistor
- removed R14: 330R, Resistor_THT:R_Axial_DIN0207_L6.3mm_D2.5mm_P10.16mm_Horizontal, symbol PCM_SL_Resistors:Resistor
- removed R15: 1R±5%, Resistor_THT:R_Axial_DIN0414_L11.9mm_D4.5mm_P25.40mm_Horizontal, symbol PCM_SL_Resistors:Resistor
- removed R16: 20R, Resistor_THT:R_Axial_DIN0207_L6.3mm_D2.5mm_P10.16mm_Horizontal, symbol PCM_SL_Resistors:Resistor
- removed R17: 464R, Resistor_THT:R_Axial_DIN0207_L6.3mm_D2.5mm_P2.54mm_Vertical, symbol PCM_SL_Resistors:Resistor
- removed R18: 464R, Resistor_THT:R_Axial_DIN0207_L6.3mm_D2.5mm_P7.62mm_Horizontal, symbol PCM_SL_Resistors:Resistor
- removed R19: 330R, Resistor_THT:R_Axial_DIN0207_L6.3mm_D2.5mm_P7.62mm_Horizontal, symbol PCM_SL_Resistors:Resistor
- removed R2, R3: 5K1, Resistor_THT:R_Axial_DIN0207_L6.3mm_D2.5mm_P10.16mm_Horizontal, symbol PCM_SL_Resistors:Resistor
- removed R4: 1K, Potentiometer_THT:Potentiometer_Bourns_3296W_Vertical, symbol Device:R_Trim
- removed R8: 10K, Resistor_THT:R_Axial_DIN0207_L6.3mm_D2.5mm_P10.16mm_Horizontal, symbol PCM_SL_Resistors:Resistor
- removed RGB_LED1: RGB_LED, TerminalBlock_Phoenix:TerminalBlock_Phoenix_MPT-0,5-4-2.54_1x04_P2.54mm_Horizontal, symbol Device:LED_KRGB
- removed RV1, RV2: 50K, PCM_SL_Devices:potentiometer_3362P, symbol Device:R_Potentiometer_Trim
- removed SERIAL1: 1x2, Connector_PinSocket_2.54mm:PinSocket_1x02_P2.54mm_Vertical, symbol PCM_SL_Pin_Headers:PINHD_1x2_Male
- removed SW1: RESET, Button_Switch_THT:SW_PUSH_6mm, symbol Switch:SW_Push
- removed SW2: Horizontal, TerminalBlock_Phoenix:TerminalBlock_Phoenix_MPT-0,5-2-2.54_1x02_P2.54mm_Horizontal_RAW, symbol Switch:SW_Push
- removed SW3: Vertical, TerminalBlock_Phoenix:TerminalBlock_Phoenix_MPT-0,5-2-2.54_1x02_P2.54mm_Horizontal_RAW, symbol Switch:SW_Push
- removed TSV1: BZW06-5V8, Diode_THT:D_DO-15_P12.70mm_Horizontal, symbol Diode:1N62xxA
- removed TSV2: 1N5908, Diode_THT:D_DO-15_P12.70mm_Horizontal, symbol Diode:1N62xxA
- removed U1: ATmega328-P, Package_DIP:DIP-28_W7.62mm_Socket, symbol MCU_Microchip_ATmega:ATmega328-P
- removed U2, U3, U4, U5: TPIC6B595N, Package_DIP:DIP-20_W7.62mm_Socket_With_IC, symbol SIPO_Register_TPIC6B595N:TPIC6B595N
- removed Y1: 16MHz±20ppm, Crystal:Crystal_HC49-4H_Vertical, symbol PCM_SL_Devices:Crystal_8MHz
Connections:
- no-connect marks 1 -> 0
Other:
- added sheet Bloková Schéma (blokova_schema.kicad_sch)
- added sheet Hlavná Schéma (schema.kicad_sch)
- note removed: ""Bleeding" resistor for discharging the capacitors when power is switched off."
- note removed: "Brightness regulation (PWM)"
- note removed: "CL = (C1 * C2) / (C1 + C2) + Cstray C1 = C2 = 2CL + 2Cstray pre CL = 30pF; Cstray = 5pF => C1 = C2 = 70pF"
- note removed: "Externý pull-up rezistor aby sme zabránili nechcenému resetovaniu."
- note removed: "I = 5V / 10K = 500uA P = 5V * 500uA = 2,5mW"
- note removed: "In-circuit Serial Programmer (ICSP) Bus (standard AVR layout)"
- note removed: "Indikátor synchronizácie"
- note removed: "Keďže existuje veľa roznych verzií modulov pre príjimanie signálu DCF77 a väčšina sa lýši len poradím pinov prípadne veľkosťou napájacieho napätia (3V3/5V), potrebujeme flexibilné zapojenie, ktoré bude podporovať všetky tieto moduly. V našom prípade to riešime cez 4-pinovú svorkovnicu, ktorej káble sa dajú poprehadzovať podľa potreby."
- note removed: "MCU + Controls"
- note removed: "Modul zapojenia DS3231 SMD čipu so zabudovanou batériou. Chybovosť čipu okolo ~2ppm prvých 5 rokov, takže max. odchylka ~60 s za rok."
- note removed: "Napájanie a ovládanie modulu príjimača"
- note removed: "Napätie (podľa meraní): R: 1V72 - 1V92 G/B: 2V48 - 3V Maximálny prúd pre farbu: 5mA"
- note removed: "Numitron Display (4xIV-9)"
- note removed: "Ochrana proti opačnej polarite. Samotné TSV diódy pri opačnej polarite (priepustný smer) sa chovajú ako normálne diódy (teda Uf = ~0.6V)."
- note removed: "Panel mount power connector - USB Type C"
- note removed: "Piny PON a OUT vieme zmeniť v softvéri."
- note removed: "Podľa datasheetu majú byť C2 a C4 rovnaké. Pod kryštáľom nemajú byť žiadne iné spoje ani liata meď."
- note removed: "Podľa datasheetu piny NC nemajú žiadne interné prepojenie v čipe a mali by byť pripojené ku GND pre lepšiu distribúciu tepla."
- note removed: "Pojistka môže byť montovaná aj na krabičke. Nemalo by byť treba ju meniť, takže to asi nie je treba."
- note removed: "Power supply"
- note removed: "Príjimač signálu atomových hodín"
- note removed: "Pull-up rezistor zaistí východzí 3.3V HIGH stav."
- note removed: "RG = RB = (5V-2V48)/5*10^-3A = 544 (464) RR = (5V-1V72)/5*10^-3A = 656 (619) * Zaokrúhlene na najbližšiu bežnú hodnotu."
- note removed: "RGB LED-ka bude na panely."
- note removed: "RTC"
- note removed: "Regulácia prúdu pomocou trimra podľa potreby pripojených záťaží."
- note removed: "Schottkyho dióda zábrani 5V HIGH stavu z MCU aby poškodil 3V3 modul, v prípade chyby v sofvéri."
- note removed: "Screw terminal for VBUS and GND from the USB-C receptacle."
- note removed: "Senzor prúdového odberu displeja"
- note removed: "Softvérovo kontrolované indikačná RGB LED-ka pre DCF77 modul. Všetky farby by mali byť cez PWM."
- note removed: "Upravovanie max. jasu RGB diódy."
- note removed: "Voľba medzi +5V a +3V3 pomocou mostíkovej prepojky."
- note removed: "Zapojenie modulu príjimača"
- note removed: "Zbernica pre seriovú komunikáciu."
- note removed: "Zdroj Napätia 3V3"
