File: numeri-iv9-hodiny.kicad_pcb (KiCad board)
At the start: 2 copper layers, 150 x 50 mm, 60 parts, among them J1 USB-C, J3 2x3, Q1 BC547, SW1 RESET, SW2 Horizontal, SW3 Vertical, U1 LM2596T-5, U2 ATtiny24A-PU, U3 TPIC6B595N, Y1 6MHz

Commit message: Pridaný kód firmwaru + úpravy schéma a DPS s anglickým prekladom.
Parts:
- removed C2: 470uF_25V, Capacitor_THT:CP_Radial_D8.0mm_P3.50mm
- removed C3, C4: 1000uF, Capacitor_THT:CP_Radial_D10.0mm_P5.00mm
- removed D6, D7, D8: 1N5817, Diode_THT:D_DO-41_SOD81_P10.16mm_Horizontal
- removed G***: LOGO, hodiny:logo
- removed H_:__1, _H:__1, __:M_1, __:_M1: IV-9, Connector_PinSocket_2.54mm:PinSocket_1x04_P2.54mm_Vertical
- removed J1: USB-C, TerminalBlock_Phoenix:TerminalBlock_Phoenix_PT-1,5-2-5.0-H_1x02_P5.00mm_Horizontal
- removed L2: 33uH, Inductor_THT:L_CommonMode_Toroid_Vertical_L19.3mm_W10.8mm_Px6.35mm_Py15.24mm_Bourns_8100
- removed Q1: BC547, Package_TO_SOT_THT:TO-92_Inline
- removed R1, R2: 10k, Resistor_THT:R_Axial_DIN0207_L6.3mm_D2.5mm_P10.16mm_Horizontal
- removed the REF** at (242.0, 58.0)
- removed the REF** at (242.0, 92.0)
- removed the REF** at (108.0, 58.0)
- removed the REF** at (108.0, 92.0)
- removed SW3: Vertical, TerminalBlock_Phoenix:TerminalBlock_Phoenix_MKDS-1,5-2_1x02_P5.00mm_Horizontal
- removed TVS1: P6KE250A, Diode_THT:D_DO-41_SOD81_P10.16mm_Horizontal
- removed U1: LM2596T-5, Package_TO_SOT_THT:TO-220-5_P3.4x3.7mm_StaggerOdd_Lead3.8mm_Vertical
- removed U3: TPIC6B595N, Package_DIP:DIP-20_W7.62mm_Socket
- added D2: 1N5817, Diode_THT:D_DO-41_SOD81_P10.16mm_Horizontal, F.Cu at (56.6, 53.9)
- added D3: 1N5817, Diode_THT:D_DO-41_SOD81_P10.16mm_Horizontal, F.Cu at (56.6, 58.1)
- added H1: IV-9, Connector_PinHeader_1.00mm:PinHeader_1x05_P1.00mm_Vertical, F.Cu at (120.7, 98.3)
- added H2: IV-9, VacuumTubes:IV-9, F.Cu at (48.9, 62.3)
- added J2: USB-C, TerminalBlock_Phoenix:TerminalBlock_Phoenix_PT-1,5-2-5.0-H_1x02_P5.00mm_Horizontal, F.Cu at (58.2, 65.2)
- added M1: IV-9, VacuumTubes:IV-9, F.Cu at (48.9, 73.9)
- added M2: IV-9, VacuumTubes:IV-9, F.Cu at (48.9, 85.6)
- added REF**: MountingHole_3.2mm_M3, MountingHole:MountingHole_3.2mm_M3, F.Cu at (232.8, 121.0)
- added REF**: MountingHole_3.2mm_M3, MountingHole:MountingHole_3.2mm_M3, F.Cu at (94.9, 83.5)
- added REF**: MountingHole_3.2mm_M3, MountingHole:MountingHole_3.2mm_M3, F.Cu at (94.9, 121.0)
- added REF**: MountingHole_3.2mm_M3, MountingHole:MountingHole_3.2mm_M3, F.Cu at (232.8, 83.5)
- added TSV1: BZW06-5V8, Diode_THT:D_DO-201AE_P15.24mm_Horizontal, F.Cu at (56.8, 48.3)
- C1: value 100uF -> 470uF; footprint Capacitor_THT:CP_Radial_D5.0mm_P2.00mm -> Capacitor_THT:CP_Radial_D8.0mm_P3.50mm
- C13: value 100nF -> 100n
- C16: value 100n -> 10uF; footprint Capacitor_THT:C_Disc_D3.0mm_W2.0mm_P2.50mm -> Capacitor_THT:CP_Radial_D5.0mm_P2.00mm
- C17: value 100n -> 100nF
- C6: value 470uF_10V -> 100uF; footprint Capacitor_THT:CP_Radial_D8.0mm_P3.50mm -> Capacitor_THT:CP_Radial_D5.0mm_P2.00mm
- C9: value 10uF -> 100nF; footprint Capacitor_THT:CP_Radial_D5.0mm_P2.00mm -> Capacitor_THT:C_Disc_D3.0mm_W2.0mm_P2.50mm
- F1: value F1.25A/250VDC -> F1.25A
- R10: value 10k -> 2K5
- R11: value 10k -> 1K5
- R3, R4, R5, R6, R7, R8, R9: value 10k -> 10K
- SW1: value RESET -> Horizontal; footprint Button_Switch_THT:SW_PUSH_6mm -> TerminalBlock_Phoenix:TerminalBlock_Phoenix_MKDS-1,5-2_1x02_P5.00mm_Horizontal
- SW2: value Horizontal -> Vertical
- U4, U5, U6: value ~ -> TPIC6B595N
- moved R9 207.4 mm to (17.4, 124.5)
- moved R7 207.0 mm to (17.4, 116.4)
- moved D5 198.7 mm to (45.5, 130.7)
- moved R11 189.9 mm to (17.4, 132.6), turned to 0 degrees
- moved R4 189.8 mm to (17.4, 104.2), turned to 0 degrees
- moved BT1 176.5 mm to (68.3, 97.7), turned to 0 degrees
- moved R5 166.4 mm to (17.4, 108.3)
- moved R6 159.0 mm to (17.4, 112.3)
- moved SW1 155.2 mm to (55.3, 128.6)
- moved SW2 149.0 mm to (32.7, 111.5)
- moved R3 147.8 mm to (17.4, 100.2)
- moved J3 144.1 mm to (80.0, 127.0)
- moved C12 140.7 mm to (54.8, 124.8), turned to 0 degrees
- moved R10 138.5 mm to (17.4, 128.5)
- moved R8 132.7 mm to (17.4, 120.4), turned to 0 degrees
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Connections:
- net PA1/MOSI renamed PA1
- C1 pad 1: +5VBAT -> +5VREG
- C10 pad 2: +5VBAT -> Net-(U2-INT0/PB2~)
- C11 pad 2: Net-(U2-INT0/PB2~) -> Net-(U2-PA7~)
- C12 pad 2: Net-(D4-K) -> +5VREG
- C13 pad 2: Net-(U2-PA7~) -> +5VREG
- C16 pad 1: GND -> Net-(D4-K)
- C16 pad 2: +5VREG -> GND
- C17 pad 2: +5VREG -> Net-(D4-K)
- C6 pad 1: GND -> +5VBAT
- C6 pad 2: +5VREG -> GND
- C9 pad 1: Net-(D4-K) -> GND
- C9 pad 2: GND -> +5VBAT
- DCF-3850N-1 pad 3: Net-(DCF-3850N-1-OUT) -> PA0
- F1 pad 1: (no net) -> VCC
- F1 pad 2: (no net) -> +5VREG
- J3 pad 3: ~{RESET}/PB3 -> ~{RESET}
- R10 pad 1: Net-(U6-~{SRCLR}) -> Net-(D4-K)
- R11 pad 1: GND -> Net-(D5-Pad2)
- R11 pad 2: +5VREG -> PA0
- R3 pad 1: Net-(D4-K) -> GND
- R4 pad 1: Net-(D5-Pad2) -> ~PA5/MISO
- R4 pad 2: Net-(Q1-E) -> +5VREG
- R5 pad 1: PA5 -> ~PA6/MOSI/SDA
- R5 pad 2: +5VREG -> +5VBAT
- R6 pad 1: ~PA6/MOSI/SDA -> Net-(U3-~{SRCLR})
- R6 pad 2: +5VBAT -> +5VREG
- R7 pad 1: Net-(U3-~{SRCLR}) -> Net-(U4-~{SRCLR})
- R8 pad 1: Net-(U4-~{SRCLR}) -> Net-(U5-~{SRCLR})
- R9 pad 1: Net-(U5-~{SRCLR}) -> Net-(U6-~{SRCLR})
- SW1 pad 1: ~{RESET}/PB3 -> Net-(U2-INT0/PB2~)
- SW2 pad 1: Net-(U2-INT0/PB2~) -> Net-(U2-PA7~)
- U2 pad 13: PA0/AREF -> PA0
- U2 pad 4: ~{RESET}/PB3 -> ~{RESET}
- U4 pad 12: unconnected-(U4-RCK-Pad12) -> PA4/SCL
- U4 pad 13: unconnected-(U4-SRCK-Pad13) -> PA3
- U4 pad 14: unconnected-(U4-DRAIN4-Pad14) -> /P6
- U4 pad 15: unconnected-(U4-DRAIN5-Pad15) -> /P7
- U4 pad 16: unconnected-(U4-DRAIN6-Pad16) -> /P8
- U4 pad 17: unconnected-(U4-DRAIN7-Pad17) -> /P9
- U4 pad 4: unconnected-(U4-DRAIN0-Pad4) -> /P2
- U4 pad 5: unconnected-(U4-DRAIN1-Pad5) -> /P3
- U4 pad 6: unconnected-(U4-DRAIN2-Pad6) -> /P4
- U4 pad 7: unconnected-(U4-DRAIN3-Pad7) -> /P5
- U4 pad 9: unconnected-(U4-~{G}-Pad9) -> ~PA6/MOSI/SDA
- U5 pad 12: unconnected-(U5-RCK-Pad12) -> PA4/SCL
- U5 pad 13: unconnected-(U5-SRCK-Pad13) -> PA3
- U5 pad 14: unconnected-(U5-DRAIN4-Pad14) -> /P6
- U5 pad 15: unconnected-(U5-DRAIN5-Pad15) -> /P7
- U5 pad 16: unconnected-(U5-DRAIN6-Pad16) -> /P8
- U5 pad 17: unconnected-(U5-DRAIN7-Pad17) -> /P9
- U5 pad 4: unconnected-(U5-DRAIN0-Pad4) -> /P2
- U5 pad 5: unconnected-(U5-DRAIN1-Pad5) -> /P3
- U5 pad 6: unconnected-(U5-DRAIN2-Pad6) -> /P4
- U5 pad 7: unconnected-(U5-DRAIN3-Pad7) -> /P5
- U5 pad 9: unconnected-(U5-~{G}-Pad9) -> ~PA6/MOSI/SDA
- U6 pad 12: unconnected-(U6-RCK-Pad12) -> PA4/SCL
- U6 pad 13: unconnected-(U6-SRCK-Pad13) -> PA3
- U6 pad 14: unconnected-(U6-DRAIN4-Pad14) -> /P6
- U6 pad 15: unconnected-(U6-DRAIN5-Pad15) -> /P7
- U6 pad 16: unconnected-(U6-DRAIN6-Pad16) -> /P8
- U6 pad 17: unconnected-(U6-DRAIN7-Pad17) -> /P9
- U6 pad 4: unconnected-(U6-DRAIN0-Pad4) -> /P2
- U6 pad 5: unconnected-(U6-DRAIN1-Pad5) -> /P3
- U6 pad 6: unconnected-(U6-DRAIN2-Pad6) -> /P4
- U6 pad 7: unconnected-(U6-DRAIN3-Pad7) -> /P5
- U6 pad 9: unconnected-(U6-~{G}-Pad9) -> ~PA6/MOSI/SDA
Routing:
- net +5VREG: track 0.00 -> 23.0 mm
- net /H1_2: track 0.00 -> 4.18 mm
- net /H1_3: track 0.00 -> 4.07 mm
- net VCC: track 0.00 -> 1.37 mm
- removed copper zone on F.Cu, net GND
Other:
- board size 150 x 50 mm -> 237.6 x 202.8 mm
- board text removed: "0"
- board text removed: "0 mm"
- board text removed: "0,0000 mm / 0,0000 mm"
- board text removed: "0,01 mm"
- board text removed: "0,02"
- board text removed: "0,035 mm"
- board text removed: "0,3000 mm"
- board text removed: "1"
- board text removed: "1,51 mm"
- board text removed: "1,6000 mm"
- board text removed: "2"
- board text removed: "239,3914 mm x 87,2047 mm"
- board text removed: "3,3"
- board text removed: "4,5"
- board text removed: "B.Cu"
- board text removed: "B.Mask"
- board text removed: "B.Paste"
- board text removed: "B.Silkscreen"
- board text removed: "Barevně"
- board text removed: "Bottom Silk Screen"
- board text removed: "Bottom Solder Mask"
- board text removed: "Bottom Solder Paste"
- board text removed: "CHARAKTERISTIKA DESKY"
- board text removed: "Celkové rozměry desky:"
- board text removed: "Dielektrika"
- board text removed: "Epsilon R"
- board text removed: "F.Cu"
- board text removed: "F.Mask"
- board text removed: "F.Paste"
- board text removed: "F.Silkscreen"
- board text removed: "FR4"
- board text removed: "Konektory na hraně karty:"
- board text removed: "Kontrola impedance:"
- board text removed: "Loss Tangent"
- board text removed: "Materiál"
- board text removed: "Min spoj/vzdálenost:"
- board text removed: "Minimální průměr díry:"
- board text removed: "Ne"
- board text removed: "None"
- board text removed: "Not specified"
- board text removed: "Název vrstvy"
- board text removed: "Pokovená hrana desky:"
- board text removed: "Povrchová úprava mědi:"
- board text removed: "Počet vrstev mědi:"
- board text removed: "Půldírové plošky:"
- board text removed: "Tloušťka (mm)"
- board text removed: "Tloušťka desky:"
- board text removed: "Top Silk Screen"
- board text removed: "Top Solder Mask"
- board text removed: "Top Solder Paste"
- board text removed: "Typ"
- board text removed: "copper"
- board text removed: "core"

Commit message: Veľké pokroky pri navrhu DPS.
Parts:
- removed R4: 10K, Resistor_THT:R_Axial_DIN0207_L6.3mm_D2.5mm_P10.16mm_Horizontal
- removed REF** (x4): MountingHole_3.2mm_M3, MountingHole:MountingHole_3.2mm_M3
- added R12: 10K, Resistor_THT:R_Axial_DIN0207_L6.3mm_D2.5mm_P10.16mm_Horizontal, F.Cu at (158.5, 109.4)
- added U3: TPIC6B595N, Package_DIP:DIP-20_W7.62mm_Socket, F.Cu at (206.7, 113.6)
- C1: value 470uF -> 4,7uF
- C12, C13, C14, C15: value 100n -> 100nF
- C6: value 100uF -> 3,3uF
- D2, D3: value 1N5817 -> 1N5822
- D5: footprint LED_THT:LED_D5.0mm -> TerminalBlock_Phoenix:TerminalBlock_Phoenix_MPT-0,5-2-2.54_1x02_P2.54mm_Horizontal
- DCF-3850N-1: footprint Connector_PinHeader_2.54mm:PinHeader_1x04_P2.54mm_Vertical -> Connector_PinSocket_2.54mm:PinSocket_1x04_P2.54mm_Vertical
- H1: footprint Connector_PinHeader_1.00mm:PinHeader_1x05_P1.00mm_Vertical -> VacuumTubes:IV-9_External_Socket_Asymetric
- H2, M1, M2: footprint VacuumTubes:IV-9 -> VacuumTubes:IV-9_External_Socket_Asymetric
- SW1, SW2: footprint TerminalBlock_Phoenix:TerminalBlock_Phoenix_MKDS-1,5-2_1x02_P5.00mm_Horizontal -> TerminalBlock_Phoenix:TerminalBlock_Phoenix_MPT-0,5-2-2.54_1x02_P2.54mm_Horizontal
- moved F1 201.5 mm to (232.5, 113.4), turned to 90 degrees
- moved R6 193.5 mm to (210.2, 95.1), turned to 90 degrees
- moved R7 177.9 mm to (194.0, 95.0), turned to 90 degrees
- moved R5 173.0 mm to (189.1, 87.0), turned to 180 degrees
- moved TSV1 172.8 mm to (224.2, 91.4), turned to -90 degrees
- moved J2 167.8 mm to (219.1, 113.0)
- moved C5 163.1 mm to (216.8, 87.5), turned to 180 degrees
- moved C12 155.3 mm to (209.9, 116.8), turned to 90 degrees
- moved H2 142.0 mm to (185.1, 102.2), turned to 180 degrees
- moved SW2 141.8 mm to (174.5, 114.0)
- moved C1 139.7 mm to (216.5, 91.7), turned to -90 degrees
- moved R8 133.9 mm to (149.0, 95.7), turned to 90 degrees
- moved C13 132.0 mm to (192.1, 116.8), turned to 90 degrees
- moved R9 117.4 mm to (131.2, 95.6), turned to 90 degrees
- moved C7 112.7 mm to (166.1, 92.7)
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Connections:
- net Net-(D4-K) renamed +3.3V
- net PA0 renamed OUT
- net PA1 renamed ~{PON}
- C10 pad 2: Net-(U2-INT0/PB2~) -> MISO/HBTN
- C11 pad 2: Net-(U2-PA7~) -> VBTN
- H1 pad 5: /P5 -> /H1_5
- H2 pad 2: /P2 -> /H2_2
- H2 pad 3: /P3 -> /H2_3
- H2 pad 4: /P4 -> /H2_4
- H2 pad 5: /P5 -> /H2_5
- H2 pad 6: /P6 -> /H2_6
- H2 pad 7: /P7 -> /H2_7
- H2 pad 8: /P8 -> /H2_8
- H2 pad 9: /P9 -> /H2_9
- J3 pad 4: PA4/SCL -> ADC/SCL
- J3 pad 5: ~PA6/MOSI/SDA -> MOSI/SRCK
- J3 pad 6: ~PA5/MISO -> MISO/HBTN
- M1 pad 2: /P2 -> /M1_2
- M1 pad 3: /P3 -> /M1_3
- M1 pad 4: /P4 -> /M1_4
- M1 pad 5: /P5 -> /M1_5
- M1 pad 6: /P6 -> /M1_6
- M1 pad 7: /P7 -> /M1_7
- M1 pad 8: /P8 -> /M1_8
- M1 pad 9: /P9 -> /M1_9
- M2 pad 2: /P2 -> /M2_2
- M2 pad 3: /P3 -> /M2_3
- M2 pad 4: /P4 -> /M2_4
- M2 pad 5: /P5 -> /M2_5
- M2 pad 6: /P6 -> /M2_6
- M2 pad 7: /P7 -> /M2_7
- M2 pad 8: /P8 -> /M2_8
- M2 pad 9: /P9 -> /M2_9
- R5 pad 1: ~PA6/MOSI/SDA -> ~{G}~
- SW1 pad 1: Net-(U2-INT0/PB2~) -> MISO/HBTN
- SW2 pad 1: Net-(U2-PA7~) -> VBTN
- U2 pad 10: PA3 -> VBTN
- U2 pad 11: PA2 -> SER_IN
- U2 pad 5: Net-(U2-INT0/PB2~) -> ~{G}~
- U2 pad 6: Net-(U2-PA7~) -> RCK
- U2 pad 7: ~PA6/MOSI/SDA -> MOSI/SRCK
- U2 pad 8: ~PA5/MISO -> MISO/HBTN
- U2 pad 9: PA4/SCL -> ADC/SCL
- U4 pad 12: PA4/SCL -> RCK
- U4 pad 13: PA3 -> MOSI/SRCK
- U4 pad 14: /P6 -> /H2_6
- U4 pad 15: /P7 -> /H2_7
- U4 pad 16: /P8 -> /H2_8
- U4 pad 17: /P9 -> /H2_9
- U4 pad 4: /P2 -> /H2_2
- U4 pad 5: /P3 -> /H2_3
- U4 pad 6: /P4 -> /H2_4
- U4 pad 7: /P5 -> /H2_5
- U4 pad 9: ~PA6/MOSI/SDA -> ~{G}~
- U5 pad 12: PA4/SCL -> RCK
- U5 pad 13: PA3 -> MOSI/SRCK
- U5 pad 14: /P6 -> /M1_6
- U5 pad 15: /P7 -> /M1_7
- U5 pad 16: /P8 -> /M1_8
- U5 pad 17: /P9 -> /M1_9
- U5 pad 4: /P2 -> /M1_2
- U5 pad 5: /P3 -> /M1_3
- U5 pad 6: /P4 -> /M1_4
- U5 pad 7: /P5 -> /M1_5
- U5 pad 9: ~PA6/MOSI/SDA -> ~{G}~
- U6 pad 12: PA4/SCL -> RCK
- U6 pad 13: PA3 -> MOSI/SRCK
- U6 pad 14: /P6 -> /M2_6
- U6 pad 15: /P7 -> /M2_7
- U6 pad 16: /P8 -> /M2_8
- U6 pad 17: /P9 -> /M2_9
- U6 pad 4: /P2 -> /M2_2
- U6 pad 5: /P3 -> /M2_3
- U6 pad 6: /P4 -> /M2_4
- U6 pad 7: /P5 -> /M2_5
- U6 pad 9: ~PA6/MOSI/SDA -> ~{G}~
Routing:
- net +5VREG: track 23.0 -> 409.3 mm
- net MOSI/SRCK: track 0.00 -> 115.2 mm
- net +5VBAT: track 0.00 -> 110.0 mm
- net ~{G}~: track 0.00 -> 104.3 mm
- net RCK: track 0.00 -> 89.9 mm
- net Net-(U4-SER_OUT): track 0.00 -> 39.8 mm
- net Net-(BT1-+): track 0.00 -> 27.3 mm
- net MISO/HBTN: track 0.00 -> 23.3 mm, vias 0 -> 2
- net +3.3V: track 0.00 -> 21.1 mm
- net OUT: track 0.00 -> 21.0 mm, vias 0 -> 2
- net VBTN: track 0.00 -> 18.8 mm
- net Net-(U2-PB1/XTAL2): track 0.00 -> 11.8 mm
- net ADC/SCL: track 0.00 -> 11.1 mm, vias 0 -> 2
- net Net-(U2-PB0/XTAL1): track 0.00 -> 10.7 mm
- net Net-(U3-SER_OUT): track 0.00 -> 10.2 mm
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Other:
- board size 237.6 x 202.8 mm -> 149.9 x 49.5 mm

Commit message: Pomerne velke zmeny a prehodnotenia zakladnych veci.
Parts:
- removed C1: 4,7uF, Capacitor_THT:CP_Radial_D8.0mm_P3.50mm
- removed R11: 1K5, Resistor_THT:R_Axial_DIN0207_L6.3mm_D2.5mm_P10.16mm_Horizontal
- added C2: 4.7uF, Capacitor_THT:CP_Radial_D5.0mm_P2.00mm, F.Cu at (102.9, 118.1)
- added EM2S1: DCF77, Connector_PinSocket_2.54mm:PinSocket_1x04_P2.54mm_Vertical, F.Cu at (221.8, 117.6)
- added MASD-S-R1: DCF77, Connector_PinSocket_2.54mm:PinSocket_1x04_P2.54mm_Vertical, F.Cu at (256.0, 77.4)
- added R13: 10K, Resistor_THT:R_Axial_DIN0207_L6.3mm_D2.5mm_P5.08mm_Vertical, F.Cu at (156.7, 90.8)
- added R4: 50K, PCM_SL_Devices:potentiometer_3362P, F.Cu at (221.8, 110.8)
- added REF**: MountingHole_3.2mm_M3, MountingHole:MountingHole_3.2mm_M3, F.Cu at (235.5, 86.4)
- added REF**: MountingHole_3.2mm_M3, MountingHole:MountingHole_3.2mm_M3, F.Cu at (91.6, 85.5)
- added REF**: MountingHole_3.2mm_M3, MountingHole:MountingHole_3.2mm_M3, F.Cu at (235.5, 118.0)
- added REF**: MountingHole_3.2mm_M3, MountingHole:MountingHole_3.2mm_M3, F.Cu at (91.6, 118.0)
- added TSV2: BZW06-5V8, Diode_THT:D_DO-201AE_P15.24mm_Horizontal, F.Cu at (102.9, 113.0)
- C8: moved to B.Cu
- R12, R5: footprint Resistor_THT:R_Axial_DIN0207_L6.3mm_D2.5mm_P10.16mm_Horizontal -> Resistor_THT:R_Axial_DIN0207_L6.3mm_D2.5mm_P5.08mm_Vertical
- R3: footprint Resistor_THT:R_Axial_DIN0207_L6.3mm_D2.5mm_P10.16mm_Horizontal -> Resistor_THT:R_Axial_DIN0207_L6.3mm_D2.5mm_P2.54mm_Vertical
- moved C17 174.4 mm to (271.6, 66.1), turned to 180 degrees
- moved DCF-3850N-1 159.4 mm to (256.0, 72.8)
- moved F1 140.6 mm to (93.7, 90.9), turned to -90 degrees
- moved BT1 139.5 mm to (234.1, 101.9)
- moved D2 119.7 mm to (228.5, 95.1)
- moved D3 119.1 mm to (228.5, 99.3)
- moved J2 116.1 mm to (104.8, 92.7), turned to 90 degrees
- moved TSV1 115.7 mm to (110.5, 113.0), turned to 90 degrees
- moved C16 115.3 mm to (219.2, 90.6), turned to 0 degrees
- moved C5 111.8 mm to (109.2, 118.1)
- moved D4 109.3 mm to (218.3, 103.6), turned to 0 degrees
- moved R10 101.5 mm to (214.4, 94.5)
- moved J3 57.2 mm to (168.9, 117.2), turned to 180 degrees
- moved R5 54.2 mm to (135.1, 92.2), turned to 90 degrees
- moved C6 40.6 mm to (117.4, 74.9), turned to 0 degrees
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Connections:
- net VCC renamed VBUS
- J3 pad 1: +5VBAT -> GND
- J3 pad 2: GND -> ~{RESET}
- J3 pad 3: ~{RESET} -> MOSI/SRCK
- J3 pad 5: MOSI/SRCK -> +5VBAT
Routing:
- net +5VREG: track 409.3 -> 255.9 mm
- net +5VBAT: track 110.0 -> 47.6 mm
- net Net-(BT1-+): track 27.3 -> 0.00 mm
- net ADC/SCL: track 11.1 -> 33.9 mm, vias 2 -> 0
- net +3.3V: track 21.1 -> 0.00 mm
- net OUT: track 21.0 -> 2.63 mm, vias 2 -> 1
- net ~{G}~: track 104.3 -> 89.1 mm
- net Net-(D5-Pad2): track 10.1 -> 0.00 mm
- net MOSI/SRCK: track 115.2 -> 123.4 mm
- net MISO/HBTN: track 23.3 -> 29.1 mm, vias 2 -> 0
- net ~{RESET}: track 5.66 -> 11.2 mm, vias 2 -> 0
- net VBTN: track 18.8 -> 24.1 mm
- net Net-(U2-PB1/XTAL2): track 11.8 -> 7.55 mm
- net VBUS: track 8.53 -> 12.4 mm
- net ~{PON}: track 5.12 -> 2.63 mm, vias 2 -> 1
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- added copper zone on B.Cu, net (none)
Other:
- board size 149.9 x 49.5 mm -> 149.9 x 38.5 mm
