File: test.kicad_pcb (KiCad board)
At the start: 2 copper layers, 172 x 50 mm, 76 parts, among them J2 Screw_Terminal_01x04, J3 USB-C, J4 PINHD_1x3_Female, J5 HW-084, J6 2x3, J7 1x2, Q1 BC557, Q2 BC557, SW1 RESET, SW2 Horizontal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

Commit message: Prvá iterácia.
Parts:
- removed the G*** at (92.2, 87.8)
- removed the G*** at (108.0, 76.2)
- removed the REF** at (130.0, 111.0)
- removed the REF** at (149.0, 105.5)
- removed the REF** at (158.0, 111.0)
- added C18: 4u7, Capacitor_THT:C_Disc_D6.0mm_W2.5mm_P5.00mm, F.Cu at (147.2, 109.2)
- added C19: 1uF, Capacitor_THT:C_Disc_D6.0mm_W2.5mm_P5.00mm, F.Cu at (211.5, 109.0)
- added G***: LOGO, LOGO, F.Cu at (91.5, 87.2)
- added G***: LOGO, LOGO, F.Cu at (112.5, 77.0)
- added Q3: BC547, Package_TO_SOT_THT:TO-92_Inline, F.Cu at (176.5, 111.3)
- added R20: 10R, Resistor_THT:R_Axial_DIN0207_L6.3mm_D2.5mm_P7.62mm_Horizontal, F.Cu at (214.2, 82.8)
- added R23: 10K, Resistor_THT:R_Axial_DIN0207_L6.3mm_D2.5mm_P10.16mm_Horizontal, F.Cu at (105.0, 103.5)
- added REF**: OSHW-Symbol_6.7x6mm_SilkScreen, Symbol:OSHW-Symbol_6.7x6mm_SilkScreen, F.Cu at (186.6, 74.8)
- added REF**: WEEE-Logo_4.2x6mm_SilkScreen, Symbol:WEEE-Logo_4.2x6mm_SilkScreen, F.Cu at (75.2, 112.0)
- D1: footprint Diode_THT:D_A-405_P10.16mm_Horizontal -> Diode_THT:D_DO-41_SOD81_P12.70mm_Horizontal
- F1: value F1A25 -> F1A25/F900mA
- J2: footprint TerminalBlock_Phoenix:TerminalBlock_Phoenix_MPT-0,5-4-2.54_1x04_P2.54mm_Horizontal -> Connector_PinSocket_2.54mm:PinSocket_1x04_P2.54mm_Vertical
- R1, R18, R2, R8: footprint Resistor_THT:R_Axial_DIN0207_L6.3mm_D2.5mm_P10.16mm_Horizontal -> Resistor_THT:R_Axial_DIN0207_L6.3mm_D2.5mm_P7.62mm_Horizontal
- R10: value 10K -> 620R; footprint Resistor_THT:R_Axial_DIN0207_L6.3mm_D2.5mm_P10.16mm_Horizontal -> Resistor_THT:R_Axial_DIN0207_L6.3mm_D2.5mm_P7.62mm_Horizontal
- R11, R12, R15, R9: footprint Resistor_THT:R_Axial_DIN0207_L6.3mm_D2.5mm_P15.24mm_Horizontal -> Resistor_THT:R_Axial_DIN0207_L6.3mm_D2.5mm_P7.62mm_Horizontal
- R16: footprint Resistor_THT:R_Axial_DIN0414_L11.9mm_D4.5mm_P25.40mm_Horizontal -> Resistor_THT:R_Axial_DIN0414_L11.9mm_D4.5mm_P20.32mm_Horizontal
- R17: value 20R -> 27R; footprint Resistor_THT:R_Axial_DIN0207_L6.3mm_D2.5mm_P15.24mm_Horizontal -> Resistor_THT:R_Axial_DIN0207_L6.3mm_D2.5mm_P10.16mm_Horizontal
- R19: footprint Resistor_THT:R_Axial_DIN0207_L6.3mm_D2.5mm_P2.54mm_Vertical -> Resistor_THT:R_Axial_DIN0207_L6.3mm_D2.5mm_P10.16mm_Horizontal
- RGB_LED1: footprint TerminalBlock_Phoenix:TerminalBlock_Phoenix_MPT-0,5-4-2.54_1x04_P2.54mm_Horizontal -> Connector_JST:JST_XH_B4B-XH-A_1x04_P2.50mm_Vertical
- SW2, SW3: footprint TerminalBlock_Phoenix:TerminalBlock_Phoenix_MPT-0,5-2-2.54_1x02_P2.54mm_Horizontal_RAW -> TerminalBlock_Phoenix:TerminalBlock_Phoenix_PT-1,5-2-5.0-H_1x02_P5.00mm_Horizontal
- Y1: value 16MHz±20ppm -> 16MHz±30ppm
- moved R18 102.9 mm to (214.1, 73.8), turned to 180 degrees
- moved D4 101.5 mm to (208.8, 83.4), turned to 45 degrees
- moved C11 100.5 mm to (220.5, 79.8), turned to -90 degrees
- moved J7 93.2 mm to (215.2, 88.2), turned to 90 degrees
- moved R8 64.4 mm to (187.8, 89.1)
- moved R10 60.5 mm to (165.7, 111.5), turned to 0 degrees
- moved R1 47.9 mm to (167.8, 73.8), turned to -90 degrees
- moved R12 43.5 mm to (138.5, 88.8)
- moved SW1 42.8 mm to (179.2, 77.9), turned to 180 degrees
- moved D1 41.5 mm to (122.7, 117.0), turned to 0 degrees
- moved C17 29.8 mm to (123.6, 103.5), turned to -90 degrees
- moved C6 27.3 mm to (140.8, 78.5)
- moved R11 27.0 mm to (164.5, 89.0)
- moved SW2 26.2 mm to (132.1, 73.5), turned to -90 degrees
- moved SW3 26.0 mm to (156.5, 78.5), turned to 90 degrees
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Connections:
- net Net-(TSV1-A1) renamed VBUS_FUSED
- C11 pad 2: Net-(D4-A) -> ~{RESET}
- D4 pad 2: Net-(D4-A) -> ~{RESET}
- Q1 pad 1: Net-(Q1-B) -> Net-(Q1-C)
- R1 pad 1: ~{RESET} -> Net-(R1-Pad1)
- R10 pad 1: GND -> DEC_ENA
- R10 pad 2: +5V -> Net-(Q3-B)
- R14 pad 2: Net-(Q1-B) -> Net-(Q1-C)
- R18 pad 1: Net-(D4-A) -> ~{RESET}
- R18 pad 2: ~{RESET} -> Net-(R1-Pad1)
- RV2 pad 1: Net-(R19-Pad1) -> +3V3
- RV2 pad 3: +3V3 -> Net-(R19-Pad1)
- SW1 pad 2: ~{RESET} -> Net-(R1-Pad1)
- SW3 pad 1: VBTN -> GND
- SW3 pad 2: GND -> VBTN
- U1 pad 1: Net-(D4-A) -> ~{RESET}
- U1 pad 24: unconnected-(U1-PC1-Pad24) -> DEC_ENA
- U1 pad 6: unconnected-(U1-PD4-Pad6) -> Net-(U1-PD4)
Routing:
- net SER_IN/MISO: track 15.4 -> 74.0 mm
- net LED_B/MOSI: track 2.34 -> 59.8 mm
- net Net-(R1-Pad1): track 0.00 -> 39.1 mm
- net PB5: track 44.0 -> 6.73 mm, vias 0 -> 1
- net HBTN: track 64.8 -> 100.5 mm
- net +5V_DEC: track 99.4 -> 66.3 mm, vias 0 -> 4
- net Net-(Q1-E): track 0.21 -> 27.6 mm
- net Net-(Q1-C): track 0.00 -> 24.1 mm
- net ~{PON}: track 20.0 -> 3.60 mm
- net VBTN: track 94.0 -> 81.2 mm
- net Net-(Q1-B): track 4.68 -> 12.0 mm
- net +3V3: track 26.0 -> 32.9 mm
- net ~{RESET}: track 31.3 -> 37.5 mm
- net Net-(Q3-B): track 0.00 -> 6.00 mm
- net Net-(RGB_LED1-RA): track 4.98 -> 10.4 mm
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- added copper zone on B.Cu, net VBUS_FUSED
Other:
- board size 172 x 50 mm -> 160 x 50 mm
- board text added: "2025"
- board text added: "Batéria: CR2032"
- board text added: "DCF77-MODUL"
- board text added: "Hod 1"
- board text added: "Hod 10"
- board text added: "ICSP"
- board text added: "Manuál"
- board text added: "Min 1"
- board text added: "Min 10"
- board text added: "Nastavovanie napájacieho napätia pre DCF77 príjimač"
- board text added: "Podržaním vymažete EEPROM"
- board text added: "RESET"
- board text added: "RTC HW-084"
- board text added: "RX"
- board text added: "Senzorový rezistor 1Ω ± 5%"
- board text added: "TX"
- board text removed: "Diferenčný zosilňovač"
- board text removed: "NUMERI"

Commit message: Záloha pred druhým tlačením.
Parts:
- removed D4: 1N4148, Diode_THT:D_DO-35_SOD27_P7.62mm_Horizontal
- removed the G*** at (91.5, 87.2)
- removed the G*** at (112.5, 77.0)
- removed Q1, Q2: BC557, Package_TO_SOT_THT:TO-92_Inline
- removed Q3: BC547, Package_TO_SOT_THT:TO-92_Inline
- removed R17: 27R, Resistor_THT:R_Axial_DIN0207_L6.3mm_D2.5mm_P10.16mm_Horizontal
- removed R18: 330R, Resistor_THT:R_Axial_DIN0207_L6.3mm_D2.5mm_P7.62mm_Horizontal
- removed the REF** at (186.6, 74.8)
- removed the REF** at (220.0, 116.5)
- removed the REF** at (68.0, 74.5)
- removed the REF** at (220.0, 74.5)
- removed the REF** at (68.0, 116.5)
- removed RV3: 1K, Potentiometer_THT:Potentiometer_Bourns_3296W_Vertical
- added C20: 1uF, Capacitor_THT:C_Disc_D6.0mm_W2.5mm_P5.00mm, F.Cu at (161.4, 118.0)
- added G***: LOGO, LOGO, F.Cu at (111.5, 77.5)
- added G***: LOGO, LOGO, F.Cu at (91.6, 87.2)
- added R21: 10R, Resistor_THT:R_Axial_DIN0207_L6.3mm_D2.5mm_P7.62mm_Horizontal, F.Cu at (164.0, 118.0)
- added R22: 10R, Resistor_THT:R_Axial_DIN0207_L6.3mm_D2.5mm_P7.62mm_Horizontal, F.Cu at (164.4, 107.2)
- added REF**: MountingHole_4.3mm_M4, MountingHole:MountingHole_4.3mm_M4, F.Cu at (219.5, 116.0)
- added REF**: MountingHole_4.3mm_M4, MountingHole:MountingHole_4.3mm_M4, F.Cu at (219.5, 75.0)
- added REF**: JUP_P10mm, PCM_SL_Jumpers:JUP_P10mm, F.Cu at (192.8, 113.5)
- added REF**: MountingHole_4.3mm_M4, MountingHole:MountingHole_4.3mm_M4, F.Cu at (68.5, 116.0)
- added REF**: MountingHole_4.3mm_M4, MountingHole:MountingHole_4.3mm_M4, F.Cu at (68.5, 75.0)
- added U6: INA219BxD, Package_SO:SOIC-8_3.9x4.9mm_P1.27mm, B.Cu at (156.0, 116.2)
- C19: value 1uF -> 100nF
- D1: footprint Diode_THT:D_DO-41_SOD81_P12.70mm_Horizontal -> Diode_THT:D_DO-41_SOD81_P7.62mm_Horizontal
- R10: value 620R -> 10K; footprint Resistor_THT:R_Axial_DIN0207_L6.3mm_D2.5mm_P7.62mm_Horizontal -> Resistor_THT:R_Axial_DIN0207_L6.3mm_D2.5mm_P5.08mm_Vertical
- R13: value 10R -> 10K; footprint Resistor_THT:R_Axial_DIN0207_L6.3mm_D2.5mm_P15.24mm_Horizontal -> Resistor_THT:R_Axial_DIN0207_L6.3mm_D2.5mm_P5.08mm_Vertical
- R14: value 330R -> 10K; footprint Resistor_THT:R_Axial_DIN0207_L6.3mm_D2.5mm_P10.16mm_Horizontal -> Resistor_THT:R_Axial_DIN0207_L6.3mm_D2.5mm_P7.62mm_Horizontal
- R2, R3, R4: moved to F.Cu
- R20: value 10R -> 620R
- moved R14 70.1 mm to (215.7, 84.6), turned to 180 degrees
- moved C19 58.0 mm to (153.6, 111.8), turned to 0 degrees
- moved R10 49.6 mm to (214.8, 104.8), turned to 180 degrees
- moved R13 14.8 mm to (209.5, 112.6)
- moved RGB_LED1 9.70 mm to (177.4, 113.6), turned to 180 degrees
- moved C11 9.27 mm to (221.1, 89.0), turned to 90 degrees
- moved R4 6.07 mm to (191.2, 109.6)
- moved R2 6.07 mm to (185.2, 109.6)
- moved R3 6.07 mm to (188.2, 109.6)
- moved D1 4.55 mm to (127.2, 116.8)
- moved REF** 4.03 mm to (75.8, 116.0)
- moved R20 3.30 mm to (217.0, 81.1), turned to 180 degrees
- moved RV1 2.90 mm to (203.5, 108.0), turned to 180 degrees
- moved C5 2.80 mm to (201.0, 102.7)
- moved C4 2.80 mm to (198.2, 106.9)
- renumbered J3 to NAPÁJANIE1, SW2 to TLACIDLO1, SW3 to TLACIDLO2
Connections:
- net VBUS renamed VCC
- net VBUS_FUSED renamed VCC_FUSED
- C11 pad 1: GND -> ~{RESET}
- C11 pad 2: ~{RESET} -> PD4
- C19 pad 2: DEC_OUT -> +5V
- J6 pad 5: +5V -> +5V_ICSP
- R1 pad 1: Net-(R1-Pad1) -> PD4
- R10 pad 1: DEC_ENA -> SCL
- R10 pad 2: Net-(Q3-B) -> +5V
- R13 pad 1: Net-(Q1-E) -> SDA
- R14 pad 1: GND -> ~{RESET}
- R14 pad 2: Net-(Q1-C) -> +5V
- R20 pad 1: ~{RESET} -> PD4
- SW1 pad 2: Net-(R1-Pad1) -> PD4
Routing:
- net PD4: track 0.00 -> 61.2 mm
- net Net-(R1-Pad1): track 39.1 -> 0.00 mm
- net +5V: track 233.3 -> 261.0 mm
- net Net-(Q1-E): track 27.6 -> 0.00 mm
- net Net-(Q1-C): track 24.1 -> 0.00 mm
- net Net-(RGB_LED1-BA): track 7.29 -> 27.4 mm
- net Net-(RGB_LED1-GA): track 9.22 -> 21.9 mm
- net +5V_DEC: track 66.3 -> 53.7 mm, vias 4 -> 3
- net ~{RESET}: track 37.5 -> 25.4 mm
- net Net-(Q1-B): track 12.0 -> 0.00 mm
- net DEC_OUT: track 16.1 -> 4.58 mm
- net Net-(U6-IN-): track 0.00 -> 9.80 mm
- net Net-(U1-PD4): track 5.24 -> 12.8 mm
- net SER_IN/MISO: track 74.0 -> 67.8 mm
- net Net-(Q3-B): track 6.00 -> 0.00 mm
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Other:
- board text added: "DCF77-PRIJÍMAČ"
- board text added: "GND"
- board text added: "HW-084"
- board text added: "Nastavovanie napájacieho napätia pre DCF77 prijímač"
- board text added: "Poistka rýchla 1A/250V 5x20mm"
- board text removed: "DCF77-MODUL"
- board text removed: "Nastavovanie napájacieho napätia pre DCF77 príjimač"
- board text removed: "Podržaním vymažete EEPROM"
- board text removed: "Pojistka 2A/250V 5x20mm"
- board text removed: "RTC HW-084"
