File: numeri-iv9-hodiny-atmega328.kicad_pcb (KiCad board)
At the start: 2 copper layers, 160 x 50 mm, 80 parts, among them J2 Screw_Terminal_01x04, J3 USB-C, J4 PINHD_1x3_Female, J5 HW-084, J6 2x3, J7 1x2, Q1 BC557, Q2 BC557, Q3 BC547, SW1 RESET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

Commit message: Zase po dlhšej dobe preventívny commit.
Parts:
- removed the REF** at (220.0, 116.5)
- removed the REF** at (68.0, 74.5)
- removed the REF** at (220.0, 74.5)
- removed the REF** at (68.0, 116.5)
- added REF**: MountingHole_4.3mm_M4, MountingHole:MountingHole_4.3mm_M4, F.Cu at (219.5, 116.0)
- added REF**: MountingHole_4.3mm_M4, MountingHole:MountingHole_4.3mm_M4, F.Cu at (219.5, 75.0)
- added REF**: MountingHole_4.3mm_M4, MountingHole:MountingHole_4.3mm_M4, F.Cu at (68.5, 116.0)
- added REF**: MountingHole_4.3mm_M4, MountingHole:MountingHole_4.3mm_M4, F.Cu at (68.5, 75.0)
- Y1: value 16MHz±30ppm -> 16MHz±20ppm
- moved REF** 4.00 mm to (75.8, 116.0)
- moved C11 1.90 mm to (221.8, 81.2), turned to 180 degrees
- moved R18 0.50 mm to (213.6, 73.8)
- renumbered J3 to NAPÁJANIE1, SW2 to TLACIDLO1, SW3 to TLACIDLO2
Routing:
- net HBTN: track 100.5 -> 95.9 mm
- net ~{RESET}: track 37.5 -> 41.0 mm
Other:
- board text added: "GND"
- board text added: "Pojistka rychlá 1A/250V 5x20mm"
- board text added: "Serial"
- board text removed: "Pojistka 2A/250V 5x20mm"

Commit message: Záloha pred druhým tlačením.
Parts:
- removed D4: 1N4148, Diode_THT:D_DO-35_SOD27_P7.62mm_Horizontal
- removed Q1, Q2: BC557, Package_TO_SOT_THT:TO-92_Inline
- removed Q3: BC547, Package_TO_SOT_THT:TO-92_Inline
- removed R17: 27R, Resistor_THT:R_Axial_DIN0207_L6.3mm_D2.5mm_P10.16mm_Horizontal
- removed R18: 330R, Resistor_THT:R_Axial_DIN0207_L6.3mm_D2.5mm_P7.62mm_Horizontal
- removed the REF** at (186.6, 74.8)
- removed RV3: 1K, Potentiometer_THT:Potentiometer_Bourns_3296W_Vertical
- added C20: 1uF, Capacitor_THT:C_Disc_D6.0mm_W2.5mm_P5.00mm, F.Cu at (161.4, 118.0)
- added R21: 10R, Resistor_THT:R_Axial_DIN0207_L6.3mm_D2.5mm_P7.62mm_Horizontal, F.Cu at (164.0, 118.0)
- added R22: 10R, Resistor_THT:R_Axial_DIN0207_L6.3mm_D2.5mm_P7.62mm_Horizontal, F.Cu at (164.4, 107.2)
- added REF**: JUP_P10mm, PCM_SL_Jumpers:JUP_P10mm, F.Cu at (192.8, 113.5)
- added U6: INA219BxD, Package_SO:SOIC-8_3.9x4.9mm_P1.27mm, B.Cu at (156.0, 116.2)
- C19: value 1uF -> 100nF
- D1: footprint Diode_THT:D_DO-41_SOD81_P12.70mm_Horizontal -> Diode_THT:D_DO-41_SOD81_P7.62mm_Horizontal
- R10: value 620R -> 10K; footprint Resistor_THT:R_Axial_DIN0207_L6.3mm_D2.5mm_P7.62mm_Horizontal -> Resistor_THT:R_Axial_DIN0207_L6.3mm_D2.5mm_P5.08mm_Vertical
- R13: value 10R -> 10K; footprint Resistor_THT:R_Axial_DIN0207_L6.3mm_D2.5mm_P15.24mm_Horizontal -> Resistor_THT:R_Axial_DIN0207_L6.3mm_D2.5mm_P5.08mm_Vertical
- R14: value 330R -> 10K; footprint Resistor_THT:R_Axial_DIN0207_L6.3mm_D2.5mm_P10.16mm_Horizontal -> Resistor_THT:R_Axial_DIN0207_L6.3mm_D2.5mm_P7.62mm_Horizontal
- R2, R3, R4: moved to F.Cu
- R20: value 10R -> 620R
- Y1: value 16MHz±20ppm -> 16MHz±30ppm
- moved R14 70.1 mm to (215.7, 84.6), turned to 180 degrees
- moved C19 58.0 mm to (153.6, 111.8), turned to 0 degrees
- moved R10 49.6 mm to (214.8, 104.8), turned to 180 degrees
- moved R13 14.8 mm to (209.5, 112.6)
- moved RGB_LED1 9.70 mm to (177.4, 113.6), turned to 180 degrees
- moved C11 7.85 mm to (221.1, 89.0), turned to 90 degrees
- moved R4 6.07 mm to (191.2, 109.6)
- moved R2 6.07 mm to (185.2, 109.6)
- moved R3 6.07 mm to (188.2, 109.6)
- moved D1 4.55 mm to (127.2, 116.8)
- moved R20 3.30 mm to (217.0, 81.1), turned to 180 degrees
- moved RV1 2.90 mm to (203.5, 108.0), turned to 180 degrees
- moved C5 2.80 mm to (201.0, 102.7)
- moved C4 2.80 mm to (198.2, 106.9)
Connections:
- net VBUS renamed VCC
- net VBUS_FUSED renamed VCC_FUSED
- C11 pad 1: GND -> ~{RESET}
- C11 pad 2: ~{RESET} -> PD4
- C19 pad 2: DEC_OUT -> +5V
- J6 pad 5: +5V -> +5V_ICSP
- R1 pad 1: Net-(R1-Pad1) -> PD4
- R10 pad 1: DEC_ENA -> SCL
- R10 pad 2: Net-(Q3-B) -> +5V
- R13 pad 1: Net-(Q1-E) -> SDA
- R14 pad 1: GND -> ~{RESET}
- R14 pad 2: Net-(Q1-C) -> +5V
- R20 pad 1: ~{RESET} -> PD4
- SW1 pad 2: Net-(R1-Pad1) -> PD4
Routing:
- net PD4: track 0.00 -> 61.2 mm
- net Net-(R1-Pad1): track 39.1 -> 0.00 mm
- net Net-(Q1-E): track 27.6 -> 0.00 mm
- net +5V: track 233.9 -> 261.0 mm
- net Net-(Q1-C): track 24.1 -> 0.00 mm
- net Net-(RGB_LED1-BA): track 7.29 -> 27.4 mm
- net ~{RESET}: track 41.0 -> 25.4 mm
- net Net-(RGB_LED1-GA): track 9.22 -> 21.9 mm
- net +5V_DEC: track 66.3 -> 53.7 mm, vias 4 -> 3
- net Net-(Q1-B): track 12.0 -> 0.00 mm
- net DEC_OUT: track 16.1 -> 4.58 mm
- net Net-(U6-IN-): track 0.00 -> 9.80 mm
- net Net-(U1-PD4): track 5.24 -> 12.8 mm
- net SER_IN/MISO: track 74.0 -> 67.8 mm
- net Net-(Q3-B): track 6.00 -> 0.00 mm
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Other:
- board text added: "DCF77-PRIJÍMAČ"
- board text added: "Nastavovanie napájacieho napätia pre DCF77 prijímač"
- board text added: "Poistka rýchla 1A/250V 5x20mm"
- board text removed: "DCF77-MODUL"
- board text removed: "Nastavovanie napájacieho napätia pre DCF77 príjimač"
- board text removed: "Podržaním vymažete EEPROM"
- board text removed: "Pojistka rychlá 1A/250V 5x20mm"
- board text removed: "Serial"

Commit message: Úpravy stránky a firmvéru.
Parts:
- moved R12 1.02 mm to (137.5, 89.0)
- moved TLACIDLO1 1.00 mm to (131.1, 73.5)
- moved G*** 0.66 mm to (111.6, 76.8)
- moved TLACIDLO2 0.37 mm to (156.9, 78.5)
Routing:
- net SDA: track 35.0 -> 31.1 mm, vias 2 -> 1
- net SCL: track 47.3 -> 44.5 mm, vias 2 -> 1
- net Net-(U6-IN-): track 9.80 -> 8.61 mm
- net Net-(U4-~{SRCLR}): track 4.42 -> 3.24 mm
- net Net-(U1-AREF): track 4.04 -> 3.07 mm
- net Net-(U1-PD4): track 12.8 -> 11.9 mm
- net ~{PON}: track 3.73 -> 2.88 mm
- net PD4: track 61.2 -> 60.5 mm
- net Net-(R19-Pad1): track 4.50 -> 3.86 mm
- net DEC_OUT: track 4.58 -> 3.97 mm
- net +5V: track 261.0 -> 260.3 mm
- net OUT: track 3.40 -> 2.80 mm
- net +3V3: track 32.9 -> 32.3 mm
- net Net-(RGB_LED1-RA): track 16.4 -> 15.8 mm
- net +5V_DEC: track 53.7 -> 53.1 mm, vias 3 -> 0
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Other:
- board text added: "Web"
- board text removed: "Manuál"
