File: schema.kicad_sch (KiCad schematic)
At the start: 76 parts, among them J1 USB_C_Receptacle_PowerOnly_6P, J2 Screw_Terminal_01x04, J4 PINHD_1x3_Female, J5 HW-084, J6 2x3, J7 1x2, Q1 BC557, Q2 BC557, Q3 BC547, SW1 RESET, U1 ATmega328-P, U2 TPIC6B595N, U3 TPIC6B595N, U4 TPIC6B595N, U5 TPIC6B595N, Y1 16MHz±20ppm

Commit message: Záloha pred druhým tlačením.
Parts:
- removed D4: 1N4148, Diode_THT:D_DO-35_SOD27_P7.62mm_Horizontal, symbol Diode:1N4148
- removed F2: Polyfuse, symbol Device:Polyfuse
- removed Q1, Q2: BC557, Package_TO_SOT_THT:TO-92_Inline, symbol Transistor_BJT:BC557
- removed Q3: BC547, Package_TO_SOT_THT:TO-92_Inline, symbol Transistor_BJT:BC547
- removed R17: 27R, Resistor_THT:R_Axial_DIN0207_L6.3mm_D2.5mm_P10.16mm_Horizontal, symbol PCM_SL_Resistors:Resistor
- removed R18: 330R, Resistor_THT:R_Axial_DIN0207_L6.3mm_D2.5mm_P7.62mm_Horizontal, symbol PCM_SL_Resistors:Resistor
- removed RV3: 1K, Potentiometer_THT:Potentiometer_Bourns_3296W_Vertical, symbol Device:R_Potentiometer_Trim
- added C20: 1uF, Capacitor_THT:C_Disc_D6.0mm_W2.5mm_P5.00mm, symbol PCM_SL_Devices:Capacitor_NP
- added PREPÍNAČ_1: SW_DPDT_x2, symbol Switch:SW_DPDT_x2
- added R21, R22: 10R, Resistor_THT:R_Axial_DIN0207_L6.3mm_D2.5mm_P7.62mm_Horizontal, symbol PCM_SL_Resistors:Resistor
- added U6: INA219BxD, Package_SO:SOIC-8_3.9x4.9mm_P1.27mm, symbol Sensor_Energy:INA219BxD
- C19: value 1uF -> 100nF; U 25V -> 50V
- D1: footprint Diode_THT:D_DO-41_SOD81_P12.70mm_Horizontal -> Diode_THT:D_DO-41_SOD81_P7.62mm_Horizontal
- R10: value 620R -> 10K; footprint Resistor_THT:R_Axial_DIN0207_L6.3mm_D2.5mm_P7.62mm_Horizontal -> Resistor_THT:R_Axial_DIN0207_L6.3mm_D2.5mm_P5.08mm_Vertical
- R13: value 10R -> 10K; footprint Resistor_THT:R_Axial_DIN0207_L6.3mm_D2.5mm_P15.24mm_Horizontal -> Resistor_THT:R_Axial_DIN0207_L6.3mm_D2.5mm_P5.08mm_Vertical
- R14: value 330R -> 10K; footprint Resistor_THT:R_Axial_DIN0207_L6.3mm_D2.5mm_P10.16mm_Horizontal -> Resistor_THT:R_Axial_DIN0207_L6.3mm_D2.5mm_P7.62mm_Horizontal
- R20: value 10R -> 620R
- Y1: value 16MHz±20ppm -> 16MHz±30ppm
Connections:
- net +5V: now also C19.2, R10.2, R14.2, R21.2, U6.5 (VS); no longer J6.5
- net +5V_DEC: now also 1m1.1, C13.2, U2.2 (VCC), R22.1
- net DEC_ENA: no longer R10.1
- net DEC_OUT: no longer C19.2
- net GND: now also U6.1 (A1), U6.2 (A0), U6.6 (GND); no longer C11.1, R14.1
- net SCL: now also R10.1, U6.4 (SCL)
- net SDA: now also R13.1, U6.3 (SDA)
- net VBUS: now also PREPÍNAČ_1.1 (A); no longer F1.1, NAPÁJANIE1.2
- net ~{RESET}: now also C11.1, R14.1; no longer C11.2, R20.1
- net PD4: now reaches R1.1, SW1.2
- net PD4: now also C11.2, R20.1
- net VBUS_FUSED renamed VCC_FUSED
- new net: C20.1, R21.1, U6.8 (IN+)
- new net: C20.2, R22.2, U6.7 (IN-)
- new net +5V_ICSP: J6.5, PREPÍNAČ_1.3 (C)
- new net VCC: F1.1, NAPÁJANIE1.2, PREPÍNAČ_1.2 (B)
Other:
- note added: "Current_LSB = 1 / 2^15 Cal = trunc(0.04096 / ((1 / 2^15) * 1) Cal treba nahrať do kalibračného registra."
- note added: "Externý pull-up rezistor aby sme zabránili nechcenému resetovaniu. Pin má aj zabudovaný interný rezistor 30-60K aj DP filter. Bez ochrany proti ESD."
- note added: "In-circuit Serial Programmer (ICSP) Bus (štandardné rozloženie pre AVR)"
- note added: "Interné pull-up rezistory majú príliš veľké hodnoty pre I2C zbernicu."
- note added: "Každý z I/O pinov má zabudovaný voliteľný 20-50K pull-up rezistor, ktorý je možné nastaviť cez PORT register."
- note added: "Pomocou prepínača môžeme prepínať medzi zdrojom napájania. Mimo programovacieho režimu slúži ako vypínač."
- note added: "USB Typ-C Konektor na panely"
- note removed: "Externý pull-up rezistor aby sme zabránili nechcenému resetovaniu. Pin má aj zabudovaný interný rezistor 4,7K aj DP filter. Bez ochrany proti ESD."
- note removed: "In-circuit Serial Programmer (ICSP) Bus (standard AVR layout)"
- note removed: "Panel mount power connector - USB Type C"
- note removed: "Screw terminal for VBUS and GND from the USB-C receptacle."
- moved on the sheet: C11, J1, J5, NAPÁJANIE1, R1, R5, R6, SW1

Commit message: Úpravy stránky a firmvéru.
Other:
- note added: "Kondezátor pomáha zmierniť vplyv úbytku napätia na jas. Tiež by mal vykryť prudové výkyvy pri zmene segmentov."
- note added: "MCU + Ovládanie"
- note added: "Pull-up rezistor zaistí východzí 3V3/5V HIGH stav podľa nastavenia vyššie."
- note added: "Registre majú ochranu proti indukčným prechodom, spôsobeným tungstenovými vláknami numitronov. Tiež limitujú prúd na 500mA (25°C) pre každý pin, tento limit klesá zo stúpajúcou teplotou."
- note added: "Regulácia jasu pomocou PWM modulovaného ~{G} pinu. Frekvencia by mala byť od 30kHz vyššie, tak aby nerušila DCF77 prijímač."
- note added: "Svorky +IN a -IN by mali byť umiestené čo najbližšie k svorkám senzorového rezistora (Kelvinovo zapojenie inak treba počítať z odporom vodičov)."
- note removed: "Brightness regulation (PWM)"
- note removed: "MCU + Controls"
- note removed: "Pull-up rezistor zaistí východzí 3V3 HIGH stav."
- moved on the sheet: C10, C12, C18, C8, C9, F1, FB1, R23, TSV1, TSV2

Commit message: Pridaný firmware.
Parts:
- TLACIDLO1: value Horizontal -> Control; Typ Control -> (none)
- TLACIDLO2: value Vertical -> Control; Typ Control -> (none)
- U1: value ATmega328-P -> ATmega328/ATmega328P
Other:
- note added: "0"
- note added: "0x"
- note added: "4"
- note added: "Graf živostnosti tungstenových vlákien v závislosti od napájacieho napätia."
- note added: "Keďže existuje veľa rôznych verzií modulov pre príjimanie signálu DCF77 a väčšina sa lýši len poradím pinov prípadne veľkosťou napájacieho napätia (3V3/5V), potrebujeme flexibilné zapojenie, ktoré bude podporovať všetky tieto moduly. V našom prípade to riešime cez 4-pinovú svorkovnicu, ktorej káble sa dajú poprehadzovať podľa potreby."
- note added: "Mikrokontróler ako I2C master by mal mať pull-up rezistory na SDA/SCL pinoch (interné sú príliš slabé)."
- note added: "Numitronový Displej"
- note added: "Pomocou prepínača (ON-ON) môžeme prepínať medzi zdrojom napájania. Mimo programovacieho režimu slúži ako vypínač."
- note added: "Pre zníženie spotreby sa odporúča odstaviť indikačnú diódu napájania LED1 odstránením rezistora U3. V prípade, že záložná batéria nie je dobíjateľná, je potrebné odstrániť aj rezistor U4."
- note added: "Schéma zapojenia RTC modulu."
- note added: "Svorky +IN a -IN by mali byť umiestené čo najbližšie k svorkám senzorového rezistora (Kelvinovo zapojenie inak treba počítať s odporom vodičov)."
- note added: "V najhoršom prípade (každý segment odoberá 22.5mA) by mal odber jednoho plne rozsvieteného numitronu byť približne 180mA, čo je ďaleko pod limitom registrov."
- note added: "V prípade potreby môže byť vstupná kapacita za feritovým jádrom zosílená."
- note added: "Výstup modulu (OUT) bude pripojený k pinu s ADC prevodníkom aby sme podporovali aj 3.3V logiku aj 5V logiku."
- note added: "Živostnosť klasickej vláknovej žiarovky je nepriamo úmerná 13 až 14 mocnine napájacieho napätia. Teda znížením napájacieho napätia o 10% by sa mala životnosť predlžiť približne dvakrát."
- note removed: "CL = (C1 * C2) / (C1 + C2) + Cstray C1 = C2 = 2CL + 2Cstray pre CL = 30pF; Cstray = 5pF => C1 = C2 = 70pF Najbližšia štandardná hodnota: 68p"
- note removed: "Keďže existuje veľa roznych verzií modulov pre príjimanie signálu DCF77 a väčšina sa lýši len poradím pinov prípadne veľkosťou napájacieho napätia (3V3/5V), potrebujeme flexibilné zapojenie, ktoré bude podporovať všetky tieto moduly. V našom prípade to riešime cez 4-pinovú svorkovnicu, ktorej káble sa dajú poprehadzovať podľa potreby."
- note removed: "Numitron Display (4xIV-9)"
- note removed: "Pomocou prepínača môžeme prepínať medzi zdrojom napájania. Mimo programovacieho režimu slúži ako vypínač."
- note removed: "Svorky +IN a -IN by mali byť umiestené čo najbližšie k svorkám senzorového rezistora (Kelvinovo zapojenie inak treba počítať z odporom vodičov)."
- company: (none) -> ZVL Kořna
- title: (none) -> Rádiovo Riadené Numitronové Hodiny
- moved on the sheet: 10h1, 10m1, 1h1, 1m1, C1, C10, C11, C12, C13, C14, C15, C16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

Commit message: Preventívne nahratie.
Parts:
- added R17: R_Photo, symbol Device:R_Photo
Connections:
- net GND: now also R17.2
- net DEC_ENA renamed LDR
- net LDR: now also R17.1
- net DEC_OUT: no longer names the net of U1.25 (PC2)
Other:
- note added: "Snímař svetla pre kompenzáciu jasu."
