File: schema.kicad_sch (KiCad schematic)
At the start: 74 parts, among them J1 USB_C_Receptacle_PowerOnly_6P, J2 Screw_Terminal_01x04, J4 PINHD_1x3_Female, J5 HW-084, J6 2x3, J7 1x2, SW1 RESET, U1 ATmega328/ATmega328P, U2 TPIC6B595N, U3 TPIC6B595N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

Commit message: Nove fotky.
Parts:
- U2, U3, U4, U5: value TPIC6B595N -> TPIC6B595N/TPIC6595N
Other:
- note added: "Podľa datasheetu majú byť kondezátory krištála rovnaké. Pod kryštálom nemajú byť žiadne iné spoje ani liata meď."
- note removed: "Podľa datasheetu majú byť C2 a C4 rovnaké. Pod kryštáľom nemajú byť žiadne iné spoje ani liata meď."

Commit message: Nové fotky a úpravy stránky.
Parts:
- R16: value 1R±5% -> 0R33
Connections:
- net SCL: no longer J6.4
- net PB5 renamed SCK/~{PON}
- net SCK/~{PON}: now also J6.4
- net PD4 renamed RSTBTN
Other:
- note added: "Imax = 1 [A] Current_LSB = Imax / 2^15 Cal = trunc(0.04096 / (Current_LSB * Rshunt) Cal treba nahrať do kalibračného registra. 0,04096 - interná fixná hodnota."
- note removed: "Current_LSB = 1 / 2^15 Cal = trunc(0.04096 / ((1 / 2^15) * 1) Cal treba nahrať do kalibračného registra."
- note removed: "MCU + Ovládanie"
- note removed: "Napájanie"
- note removed: "Numitronový Displej"
- note removed: "Príjimač signálu atomových hodín"
- note removed: "RTC"
- note removed: "Senzor prúdového odberu displeja"
- note removed: "USB Typ-C Konektor na panely"
- note removed: "Zdroj Napätia 3V3"
