File: export.kicad_pcb (KiCad board)
At the start: 2 copper layers, 160 x 50 mm, 77 parts, among them J2 Screw_Terminal_01x04, J4 PINHD_1x3_Female, J5 HW-084, J6 2x3, J7 1x2, SW1 RESET, U1 ATmega328-P, U2 TPIC6B595N, U3 TPIC6B595N, U4 TPIC6B595N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

Commit message: Preventívne nahratie.
Parts:
- added REF**: LED, PanelMount:LED, F.Cu at (166.5, 75.0)
- added REF**: Switch, PanelMount:Switch, F.Cu at (121.5, 75.0)
- added REF**: Button, PanelMount:Button, F.Cu at (185.5, 75.0)
- added REF**: Button, PanelMount:Button, F.Cu at (102.5, 75.0)
- added REF**: DCF77_ANTENNA_140x10mm, PanelMount:DCF77_ANTENNA_140x10mm, F.Cu at (144.5, 120.5)
Routing:
- net PB5: vias 1 -> 2
- added copper zone on B.Cu, net PB5
